Commit message: debugging gripper_controller

File: docker/cyton_ros2/src/ros2_RobotSimulation/Cyton/.ignore/cyton_gamma_300_description/cyton_gamma_300_macros.urdf.xacro (robot description, xacro)
@@ -214,5 +214,5 @@
         </link>
         <!-- Eighth motor located here -->
-        <joint name="${prefix}gripper_joint2" type="prismatic">
+        <joint name="${prefix}mimic_gripper_joint" type="prismatic">
             <parent link="${prefix}wrist_roll" />
             <child link="${prefix}gripper_finger2" />

File: docker/cyton_ros2/src/ros2_RobotSimulation/Cyton/cyton_moveit/config/cyton.ros2_control.xacro (robot description, xacro)
@@ -64,8 +64,7 @@
                 <state_interface name="velocity"/>
             </joint>
-            <joint name="gripper_joint2">
-                <command_interface name="position"/>
+            <joint name="mimic_gripper_joint">
                 <state_interface name="position">
-                  <param name="initial_value">${initial_positions['gripper_joint2']}</param>
+                  <param name="initial_value">${initial_positions['mimic_gripper_joint']}</param>
                 </state_interface>
                 <state_interface name="velocity"/>

File: docker/cyton_ros2/src/ros2_RobotSimulation/Cyton/cyton_ros2_gazebo/urdf/.ignore/cyton_gazebo.xacro (robot description, xacro)
@@ -178,5 +178,5 @@
       </joint> -->
       <!-- cyton_finger_joint2 -->
-      <!-- <joint name="gripper_joint2">
+      <!-- <joint name="mimic_gripper_joint">
         <command_interface name="position">
           <param name="min">-0.001</param>

File: docker/cyton_ros2/src/ros2_RobotSimulation/Cyton/cyton_ros2_gazebo/urdf/cyton_ignition.xacro (robot description, xacro)
@@ -182,14 +182,5 @@
       </joint>
       <!-- cyton_joint7 -->
-      <joint name="gripper_joint2">
-        <!-- <param name="initial_position">0.785</param> -->
-        <command_interface name="position">
-          <param name="min">-3.15</param> <!-- ** -3.935 -->
-          <param name="max">3.15</param> <!-- ** 2.365 -->
-        </command_interface>
-        <command_interface name="velocity">
-          <param name="min">-2.6100</param>
-          <param name="max">2.6100</param>
-        </command_interface>
+      <joint name="mimic_gripper_joint">
         <state_interface name="position"/>
         <state_interface name="velocity"/>
@@ -211,5 +202,5 @@
       </joint> -->
       <!-- cyton_finger_joint2 -->
-      <!-- <joint name="gripper_joint2">
+      <!-- <joint name="mimic_gripper_joint">
         <command_interface name="position">
           <param name="min">-0.001</param>

File: docker/cyton_ros2/src/ros2_RobotSimulation/Cyton/cyton_ros2_gazebo/urdf/cyton_macros.urdf.xacro (robot description, xacro)
@@ -292,5 +292,5 @@
         <link name="gripper_finger1">
             <visual>
-                <origin xyz="0 0 -0.033" rpy="0 0 0" />
+                <origin xyz="0 0 -0.03" rpy="0 0 0" />
                 <geometry>
                     <mesh filename="file://$(find cyton_ros2_gazebo)/meshes/visual/Gripper_Finger1.dae"/>
@@ -299,5 +299,5 @@
             </visual>
             <collision>
-                <origin xyz="0 0 -0.033" rpy="0 0 0" />
+                <origin xyz="0 0 -0.03" rpy="0 0 0" />
                 <geometry>
                     <mesh filename="file://$(find cyton_ros2_gazebo)/meshes/collision/Gripper_Finger1.stl"/>
@@ -312,5 +312,5 @@
         </link>
         <!-- Eighth motor located here -->
-        <joint name="gripper_joint2" type="prismatic">
+        <joint name="mimic_gripper_joint" type="prismatic">
             <parent link="wrist_roll" />
             <child link="gripper_finger2" />
@@ -318,10 +318,10 @@
             <dynamics damping="0.5" friction="0.5"/>
             <limit lower="-0.008" upper="0.008" effort="7.0" velocity="1.0" />
-            <!-- <mimic joint="gripper_joint" multiplier="-1"/> -->
+            <mimic joint="gripper_joint" multiplier="-1"/>
             <axis xyz="1 0 0" />
         </joint>
         <link name="gripper_finger2">
             <visual>
-                <origin xyz="0 0 -0.033" rpy="0 0 0" />
+                <origin xyz="0 0 -0.03" rpy="0 0 0" />
                 <geometry>
                     <mesh filename="file://$(find cyton_ros2_gazebo)/meshes/visual/Gripper_Finger2.dae"/>
@@ -330,5 +330,5 @@
             </visual>
             <collision>
-                <origin xyz="0 0 -0.033" rpy="0 0 0" />
+                <origin xyz="0 0 -0.03" rpy="0 0 0" />
                 <geometry>
                     <mesh filename="file://$(find cyton_ros2_gazebo)/meshes/collision/Gripper_Finger2.stl"/>

File: docker/cyton_ros2/src/ros2_RobotSimulation/Cyton/cyton_ros2_gazebo/urdf/cyton_transmission.xacro (robot description, xacro)
@@ -130,7 +130,7 @@
   </transmission>
 <!-- TODO Motor 9 in reality is motor 8, don't know solution yet -->
-  <transmission name="tran9">
+  <!-- <transmission name="tran9">
     <type>transmission_interface/SimpleTransmission</type>
-    <joint name="gripper_joint2">
+    <joint name="mimic_gripper_joint">
       <hardwareInterface>PositionJointInterface</hardwareInterface>
     </joint>
@@ -138,5 +138,5 @@
       <hardwareInterface>PositionJointInterface</hardwareInterface>
     </actuator>
-  </transmission>
+  </transmission> -->
   </xacro:macro>
 </robot>
