Commit message: gripper problem

File: docker/cyton_ros2/src/ros2_RobotSimulation/Cyton/cyton_ros2_gazebo/urdf/cyton_ignition.xacro (robot description, xacro)
@@ -188,5 +188,5 @@
       </joint>
       <!-- cyton_finger_joint1 -->
-      <!-- <joint name="joint8">
+      <joint name="joint8">
         <command_interface name="position">
           <param name="min">-0.001</param>
@@ -200,19 +200,11 @@
         <state_interface name="velocity"/>
         <state_interface name="effort"/>
-      </joint> -->
+      </joint>
       <!-- cyton_finger_joint2 -->
-      <!-- <joint name="joint9">
-        <command_interface name="position">
-          <param name="min">-0.001</param>
-          <param name="max">0.04</param>
-        </command_interface>
-        <command_interface name="velocity">
-          <param name="min">-0.3</param>
-          <param name="max">0.3</param>
-        </command_interface>
-        <state_interface name="position"/>
-        <state_interface name="velocity"/>
-        <state_interface name="effort"/>
-      </joint> -->
+      <joint name="joint9">
+        <state_interface name="position"/>
+        <state_interface name="velocity"/>
+        <state_interface name="effort"/>
+      </joint>
     </ros2_control>
     <gazebo reference="joint1">

File: docker/cyton_ros2/src/ros2_RobotSimulation/Cyton/cyton_ros2_gazebo/urdf/cyton_macros.urdf.xacro (robot description, xacro)
@@ -66,5 +66,5 @@
             <parent link="base_link" />
             <child link="joint1" />
-            <origin xyz="0 0 0.05315" rpy="0 0 1.2" />
+            <origin xyz="0 0 0.05315" rpy="0 0 0" />
             <dynamics damping="0.5" friction="0.5"/>
             <limit lower="-2.618" upper="2.618" effort="7.0" velocity="1.0" />
@@ -97,5 +97,5 @@
             <parent link="joint1" />
             <child link="joint2" />
-            <origin xyz="0 0 0.063" rpy="1.2 0 0" />
+            <origin xyz="0 0 0.063" rpy="0 0 0" />
             <dynamics damping="0.5" friction="0.5"/>
             <limit lower="-1.8326" upper="1.8326" effort="7.0" velocity="1.0" />
@@ -124,10 +124,9 @@
             </inertial>
         </link>
-        <!-- TUTAJ ODPIERDALA -->
         <!-- Third motor located here -->
         <joint name="joint3" type="revolute">
             <parent link="joint2" />
             <child link="joint3" />
-            <origin xyz="0 0 0.089" rpy="0 0 1.2" />
+            <origin xyz="0 0 0.089" rpy="0 0 0" />
             <dynamics damping="0.5" friction="0.5"/>
             <limit lower="-1.8326" upper="1.8326" effort="7.0" velocity="1.0" />
@@ -160,5 +159,5 @@
             <parent link="joint3" />
             <child link="joint4" />
-            <origin xyz="0 0 0.052" rpy="1.2 0 0" />
+            <origin xyz="0 0 0.052" rpy="0 0 0" />
             <dynamics damping="0.5" friction="0.5"/>
             <limit lower="-1.8326" upper="1.8326" effort="7.0" velocity="1.0" />
@@ -192,5 +191,5 @@
             <parent link="joint4" />
             <child link="joint5" />
-            <origin xyz="0 0 0.072" rpy="0 -1.2 0" />
+            <origin xyz="0 0 0.072" rpy="0 0 0" />
             <dynamics damping="0.5" friction="0.5"/>
             <limit lower="-1.8326" upper="1.8326" effort="7.0" velocity="1.0" />
@@ -223,5 +222,5 @@
             <parent link="joint5" />
             <child link="joint7" />
-            <origin xyz="0 0 0.0718" rpy="1.2 0 0" />
+            <origin xyz="0 0 0.0718" rpy="0 0 0" />
             <dynamics damping="0.5" friction="0.5"/>
             <limit lower="-1.8326" upper="1.8326" effort="7.0" velocity="1.0" />
@@ -254,5 +253,5 @@
             <parent link="joint7" />
             <child link="joint6" />
-            <origin xyz="0 0 0.051425" rpy="0 0 1.2" />
+            <origin xyz="0 0 0.051425" rpy="0 0 0" />
             <dynamics damping="0.5" friction="0.5"/>
             <limit lower="-2.61799" upper="2.61799" effort="7.0" velocity="1.0" />

Commit message: simulation working

File: docker/cyton_ros2/src/ros2_RobotSimulation/Cyton/cyton_ros2_gazebo/urdf/cyton_ignition.xacro (robot description, xacro)
@@ -59,5 +59,5 @@
   <ros2_control name="IgnitionSystem" type="system">
     <hardware>
-      <plugin name="ign_ros2_control/IgnitionSystem" filename="libign_hardware_plugins.so"></plugin>
+      <plugin>ign_ros2_control/IgnitionSystem</plugin>
     </hardware>
       <!-- cyton_joint1 -->

File: docker/cyton_ros2/src/ros2_RobotSimulation/Cyton/cyton_ros2_gazebo/urdf/cyton_macros.urdf.xacro (robot description, xacro)
@@ -56,5 +56,5 @@
             </collision>
             <inertial>
-                <mass value="1.0" />
+                <mass value="0.2" />
                 <origin rpy="0 0 0" xyz="0 0 0" />
                 <inertia ixx="1.1027" iyy="1.1027" izz="1.1027"
@@ -68,5 +68,5 @@
             <origin xyz="0 0 0.05315" rpy="0 0 0" />
             <dynamics damping="0.5" friction="0.5"/>
-            <limit lower="-2.618" upper="2.618" effort="1.0" velocity="1.0" />
+            <limit lower="-2.618" upper="2.618" effort="100.0" velocity="1.0" />
             <axis xyz="0 0 1" />
         </joint>
@@ -98,5 +98,5 @@
             <origin xyz="0 0 0.063" rpy="0 0 0" />
             <dynamics damping="0.5" friction="0.5"/>
-            <limit lower="-1.8326" upper="1.8326" effort="1.0" velocity="1.0" />
+            <limit lower="-1.8326" upper="1.8326" effort="100.0" velocity="1.0" />
             <axis xyz="1 0 0" />
         </joint>
@@ -128,5 +128,5 @@
             <origin xyz="0 0 0.089" rpy="0 0 0" />
             <dynamics damping="0.5" friction="0.5"/>
-            <limit lower="-1.8326" upper="1.8326" effort="1.0" velocity="1.0" />
+            <limit lower="-1.8326" upper="1.8326" effort="100.0" velocity="1.0" />
             <axis xyz="0 0 1" />
         </joint>
@@ -148,5 +148,5 @@
             </collision>
             <inertial>
-                <mass value="1.0" />
+                <mass value="0.2" />
                 <origin rpy="0 0 0" xyz="0 0 0" />
                 <inertia  ixx="0.004185745441913727" ixy="0" ixz="0"
@@ -160,5 +160,5 @@
             <origin xyz="0 0 0.052" rpy="0 0 0" />
             <dynamics damping="0.5" friction="0.5"/>
-            <limit lower="-1.8326" upper="1.8326" effort="1.0" velocity="1.0" />
+            <limit lower="-1.8326" upper="1.8326" effort="100.0" velocity="1.0" />
             <axis xyz="1 0 0" />
         </joint>
@@ -180,5 +180,5 @@
             </collision>
             <inertial>
-                <mass value="1.0" />
+                <mass value="0.2" />
                 <origin rpy="0 0 0" xyz="0 0 0" />
                 <inertia  ixx="0.0002991427484832406" ixy="0" ixz="0"
@@ -192,5 +192,5 @@
             <origin xyz="0 0 0.072" rpy="0 0 0" />
             <dynamics damping="0.5" friction="0.5"/>
-            <limit lower="-1.8326" upper="1.8326" effort="1.0" velocity="1.0" />
+            <limit lower="-1.8326" upper="1.8326" effort="100.0" velocity="1.0" />
             <axis xyz="0 -1 0" />
         </joint>
@@ -211,5 +211,5 @@
             </collision>
             <inertial>
-                <mass value="1.0" />
+                <mass value="0.2" />
                 <origin rpy="0 0 0" xyz="0 0 0" />
                 <inertia  ixx="0.004619866095305994" ixy="0" ixz="0"
@@ -223,5 +223,5 @@
             <origin xyz="0 0 0.0718" rpy="0 0 0" />
             <dynamics damping="0.5" friction="0.5"/>
-            <limit lower="-1.8326" upper="1.8326" effort="1.0" velocity="1.0" />
+            <limit lower="-1.8326" upper="1.8326" effort="100.0" velocity="1.0" />
             <axis xyz="1 0 0" />
         </joint>
@@ -242,5 +242,5 @@
             </collision>
             <inertial>
-                <mass value="1.0" />
+                <mass value="0.2" />
                 <origin rpy="0 0 0" xyz="0 0 0" />
                 <inertia  ixx="0.002306163215052582" ixy="0" ixz="0"
@@ -254,5 +254,5 @@
             <origin xyz="0 0 0.051425" rpy="0 0 1.5708" />
             <dynamics damping="0.5" friction="0.5"/>
-            <limit lower="-2.61799" upper="2.61799" effort="1.0" velocity="1.0" />
+            <limit lower="-2.61799" upper="2.61799" effort="100.0" velocity="1.0" />
             <axis xyz="0 0 1" />
         </joint>
@@ -273,5 +273,5 @@
             </collision>
             <inertial>
-                <mass value="1.0" />
+                <mass value="0.2" />
                 <origin rpy="0 0 0" xyz="0 0 0" />
                 <inertia  ixx="0.0015572863522148085" ixy="0" ixz="0"
@@ -285,5 +285,5 @@
             <origin xyz="-0.02131 0.00485 0.077225" rpy="0 0 0" />
             <dynamics damping="0.5" friction="0.5"/>
-            <limit lower="-0.001" upper="0.017" effort="1.0" velocity="1.0" />
+            <limit lower="-0.001" upper="0.017" effort="100.0" velocity="1.0" />
             <axis xyz="1 0 0" />
         </joint>
@@ -293,5 +293,5 @@
             <origin xyz="-0.05331 0.00485 0.077225" rpy="0 0 0" />
             <dynamics damping="0.5" friction="0.5"/>
-            <limit lower="-0.001" upper="0.017" effort="1.0" velocity="1.0" />
+            <limit lower="-0.001" upper="0.017" effort="100.0" velocity="1.0" />
             <axis xyz="1 0 0" />
         </joint> -->
@@ -311,5 +311,5 @@
             </collision>
             <inertial>
-                <mass value="1.0" />
+                <mass value="0.02" />
                 <origin rpy="0 0 0" xyz="0 0 0" />
                 <inertia  ixx="0.00011683333934843555" ixy="0" ixz="0"
@@ -323,5 +323,5 @@
             <origin xyz="0.0178 0.00485 0.077225" rpy="0 0 0" />
             <dynamics damping="0.5" friction="0.5"/>
-            <limit lower="-0.017" upper="0.001" effort="1.0" velocity="1.0" />
+            <limit lower="-0.017" upper="0.001" effort="100.0" velocity="1.0" />
             <mimic joint="joint8" multiplier="-1"/>
             <axis xyz="1 0 0" />
@@ -333,5 +333,5 @@
             <origin xyz="0.0498 0.00485 0.077225" rpy="0 0 0" />
             <dynamics damping="0.5" friction="0.5"/>
-            <limit lower="-0.017" upper="0.001" effort="1.0" velocity="1.0" />
+            <limit lower="-0.017" upper="0.001" effort="100.0" velocity="1.0" />
             <mimic joint="joint8" multiplier="-1"/>
             <axis xyz="1 0 0" />
@@ -352,5 +352,5 @@
             </collision>
             <inertial>
-                <mass value="1.0" />
+                <mass value="0.02" />
                 <origin rpy="0 0 0" xyz="0 0 0" />
                 <inertia  ixx="0.00011683333934843555" ixy="0" ixz="0"

Commit message: mimic_joint not working in gazebo

File: docker/cyton_ros2/src/ros2_RobotSimulation/Cyton/cyton_ros2_gazebo/urdf/cyton_ignition.xacro (robot description, xacro)
@@ -56,4 +56,9 @@
             <robot_param_node>robot_state_publisher</robot_param_node> -->
     </plugin>
+    <plugin name="${name_prefix}mimic_joint_plugin" filename="libroboticsgroup_gazebo_mimic_joint_plugin.so">
+      <joint>joint8</joint>
+      <mimicJoint>joint9</mimicJoint>
+        <multiplier>-1</multiplier>
+      </plugin>
     </gazebo>
   <ros2_control name="IgnitionSystem" type="system">

Commit message: mimic_joint added

File: docker/cyton_ros2/src/ros2_RobotSimulation/Cyton/cyton_ros2_gazebo/urdf/cyton_ignition.xacro (robot description, xacro)
@@ -56,9 +56,4 @@
             <robot_param_node>robot_state_publisher</robot_param_node> -->
     </plugin>
-    <plugin name="${name_prefix}mimic_joint_plugin" filename="libroboticsgroup_gazebo_mimic_joint_plugin.so">
-      <joint>joint8</joint>
-      <mimicJoint>joint9</mimicJoint>
-        <multiplier>-1</multiplier>
-      </plugin>
     </gazebo>
   <ros2_control name="IgnitionSystem" type="system">
@@ -187,4 +182,5 @@
       </joint>
       <joint name="joint9">
+        <param name="mimic">joint8</param>
         <state_interface name="position"/>
         <state_interface name="velocity"/>
@@ -224,5 +220,5 @@
       <material>Gazebo/Orange</material>
     </gazebo>
-    <gazebo reference="joint9">
+    <gazebo reference="joint9_mimic">
       <selfCollide>false</selfCollide>
       <material>Gazebo/Orange</material>

File: docker/cyton_ros2/src/ros2_RobotSimulation/Cyton/cyton_ros2_gazebo/urdf/cyton_macros.urdf.xacro (robot description, xacro)
@@ -318,5 +318,5 @@
         </link>
         <!-- Eighth motor located here -->
-        <joint name="joint9" type="prismatic">
+        <joint name="joint9_mimic" type="prismatic">
             <parent link="link7" />
             <child link="link9" />
