Commit message: still: "[cyton_hand_controller]: Joint name cannot be empty"

File: docker/cyton_ros2/src/ros2_RobotSimulation/Cyton/cyton_moveit/config/cyton.ros2_control.xacro (robot description, xacro)
@@ -64,10 +64,10 @@
                 <state_interface name="velocity"/>
             </joint>
-            <joint name="mimic_gripper_joint">
+            <!-- <joint name="mimic_gripper_joint">
                 <state_interface name="position">
                   <param name="initial_value">${initial_positions['mimic_gripper_joint']}</param>
                 </state_interface>
                 <state_interface name="velocity"/>
-            </joint>
+            </joint> -->
         </ros2_control>
     </xacro:macro>

Commit message: removed gripper

File: docker/cyton_ros2/src/ros2_RobotSimulation/Cyton/cyton_moveit/config/cyton.ros2_control.xacro (robot description, xacro)
@@ -8,14 +8,18 @@
               <param name="usb_port">/dev/ttyUSB0</param>
               <param name="baud_rate">1000000</param>
-              <!-- <param name="use_dummy">true</param> -->
+              <param name="use_dummy">true</param>
             </hardware>
-            <joint name="shoulder_roll_joint">
+            <!-- <joint name="shoulder_roll_joint"> -->
+            <joint name="joint1">
+                <param name="id">1</param>
                 <command_interface name="position"/>
                 <state_interface name="position">
-                  <param name="initial_value">${initial_positions['shoulder_roll_joint']}</param>
+                  <param name="initial_value">${initial_positions['joint1']}</param>
                 </state_interface>
                 <state_interface name="velocity"/>
             </joint>
-            <joint name="shoulder_pitch_joint">
+            <!-- <joint name="shoulder_pitch_joint"> -->
+            <joint name="joint2">
+                <param name="id">2</param>
                 <command_interface name="position"/>
                 <state_interface name="position">
@@ -24,5 +28,7 @@
                 <state_interface name="velocity"/>
             </joint>
-            <joint name="elbow_roll_joint">
+            <!-- <joint name="elbow_roll_joint"> -->
+            <joint name="joint3">
+                <param name="id">3</param>
                 <command_interface name="position"/>
                 <state_interface name="position">
@@ -31,5 +37,7 @@
                 <state_interface name="velocity"/>
             </joint>
-            <joint name="elbow_pitch_joint">
+            <!-- <joint name="elbow_pitch_joint"> -->
+            <joint name="joint4">
+                <param name="id">4</param>
                 <command_interface name="position"/>
                 <state_interface name="position">
@@ -38,5 +46,7 @@
                 <state_interface name="velocity"/>
             </joint>
-            <joint name="elbow_yaw_joint">
+            <!-- <joint name="elbow_yaw_joint"> -->
+            <joint name="joint5">
+                <param name="id">5</param>
                 <command_interface name="position"/>
                 <state_interface name="position">
@@ -45,5 +55,7 @@
                 <state_interface name="velocity"/>
             </joint>
-            <joint name="wrist_pitch_joint">
+            <!-- <joint name="wrist_pitch_joint"> -->
+            <joint name="joint6">
+                <param name="id">6</param>
                 <command_interface name="position"/>
                 <state_interface name="position">
@@ -52,5 +64,7 @@
                 <state_interface name="velocity"/>
             </joint>
-            <joint name="wrist_roll_joint">
+            <!-- <joint name="wrist_roll_joint"> -->
+            <joint name="joint7">
+                <param name="id">7</param>
                 <command_interface name="position"/>
                 <state_interface name="position">
@@ -59,5 +73,5 @@
                 <state_interface name="velocity"/>
             </joint>
-            <joint name="gripper_joint">
+            <!-- <joint name="gripper_joint">
                 <command_interface name="position"/>
                 <state_interface name="position">
@@ -65,5 +79,5 @@
                 </state_interface>
                 <state_interface name="velocity"/>
-            </joint>
+            </joint> -->
             <!-- <joint name="mimic_gripper_joint">
                 <state_interface name="position">

File: docker/cyton_ros2/src/ros2_RobotSimulation/Cyton/cyton_moveit/config/cyton.urdf.xacro (robot description, xacro)
@@ -6,4 +6,4 @@
     <!-- Import control_xacro -->
     <xacro:include filename="cyton.ros2_control.xacro" />
-    <xacro:cyton_ros2_control name="FakeSystem" initial_positions_file="$(arg initial_positions_file)"/>
+    <xacro:cyton_ros2_control name="DynamixelHardware" initial_positions_file="$(arg initial_positions_file)"/>
 </robot>

File: docker/cyton_ros2/src/ros2_RobotSimulation/Cyton/cyton_ros2_gazebo/urdf/cyton_ignition.xacro (robot description, xacro)
@@ -62,5 +62,6 @@
   </hardware>
       <!-- cyton_joint1 -->
-      <joint name="shoulder_roll_joint">
+      <!-- <joint name="shoulder_roll_joint"> -->
+      <joint name="joint1">
         <!-- <param name="initial_position">0.0</param> -->
         <command_interface name="position">
@@ -77,5 +78,6 @@
       </joint>
       <!-- cyton_joint2 -->
-      <joint name="shoulder_pitch_joint">
+      <!-- <joint name="shoulder_pitch_joint"> -->
+      <joint name="joint2">
         <!-- <param name="initial_position">-0.785</param> -->
         <command_interface name="position">
@@ -92,5 +94,6 @@
       </joint>
       <!-- cyton_joint3 -->
-      <joint name="elbow_roll_joint">
+      <!-- <joint name="elbow_roll_joint"> -->
+      <joint name="joint3">
         <!-- <param name="initial_position">0.0</param> -->
         <command_interface name="position">
@@ -107,5 +110,6 @@
       </joint>
       <!-- cyton_joint4 -->
-      <joint name="elbow_pitch_joint">
+      <!-- <joint name="elbow_pitch_joint"> -->
+      <joint name="joint4">
         <!-- <param name="initial_position">-2.356</param> -->
         <command_interface name="position">
@@ -122,5 +126,6 @@
       </joint>
       <!-- cyton_joint5 -->
-      <joint name="elbow_yaw_joint">
+      <!-- <joint name="elbow_yaw_joint"> -->
+      <joint name="joint5">
         <!-- <param name="initial_position">0.0</param> -->
         <command_interface name="position">
@@ -137,5 +142,6 @@
       </joint>
       <!-- cyton_joint6 -->
-      <joint name="wrist_pitch_joint">
+      <!-- <joint name="wrist_pitch_joint"> -->
+      <joint name="joint6">
         <!-- <param name="initial_position">1.5708</param> -->
         <command_interface name="position">
@@ -152,5 +158,6 @@
       </joint>
       <!-- cyton_joint7 -->
-      <joint name="wrist_roll_joint">
+      <!-- <joint name="wrist_roll_joint"> -->
+      <joint name="joint7">
         <!-- <param name="initial_position">0.785</param> -->
         <command_interface name="position">
@@ -167,48 +174,19 @@
       </joint>
       <!-- cyton_joint7 -->
-      <joint name="gripper_joint">
-        <!-- <param name="initial_position">0.785</param> -->
-        <command_interface name="position">
-          <param name="min">-3.15</param> <!-- ** -3.935 -->
-          <param name="max">3.15</param> <!-- ** 2.365 -->
-        </command_interface>
-        <command_interface name="velocity">
-          <param name="min">-2.6100</param>
-          <param name="max">2.6100</param>
-        </command_interface>
-        <state_interface name="position"/>
-        <state_interface name="velocity"/>
-        <state_interface name="effort"/>
-      </joint>
+      <!-- <joint name="gripper_joint">
+        <command_interface name="position">
+          <param name="min">-3.15</param>
+          <param name="max">3.15</param>
+        </command_interface>
+        <command_interface name="velocity">
+          <param name="min">-2.6100</param>
+          <param name="max">2.6100</param>
+        </command_interface>
+        <state_interface name="position"/>
+        <state_interface name="velocity"/>
+        <state_interface name="effort"/>
+      </joint> -->
       <!-- cyton_joint7 -->
-      <joint name="mimic_gripper_joint">
-        <state_interface name="position"/>
-        <state_interface name="velocity"/>
-        <state_interface name="effort"/>
-      </joint>
-      <!-- cyton_finger_joint1 -->
-      <!-- <joint name="gripper_joint">
-        <command_interface name="position">
-          <param name="min">-0.001</param>
-          <param name="max">0.04</param>
-        </command_interface>
-        <command_interface name="velocity">
-          <param name="min">-0.3</param>
-          <param name="max">0.3</param>
-        </command_interface>
-        <state_interface name="position"/>
-        <state_interface name="velocity"/>
-        <state_interface name="effort"/>
-      </joint> -->
-      <!-- cyton_finger_joint2 -->
       <!-- <joint name="mimic_gripper_joint">
-        <command_interface name="position">
-          <param name="min">-0.001</param>
-          <param name="max">0.04</param>
-        </command_interface>
-        <command_interface name="velocity">
-          <param name="min">-0.3</param>
-          <param name="max">0.3</param>
-        </command_interface>
         <state_interface name="position"/>
         <state_interface name="velocity"/>
@@ -244,5 +222,5 @@
       <material>Gazebo/Orange</material>
     </gazebo>
-    <gazebo reference="gripper_finger1">
+    <!-- <gazebo reference="gripper_finger1">
       <selfCollide>false</selfCollide>
       <material>Gazebo/Orange</material>
@@ -251,5 +229,5 @@
       <selfCollide>false</selfCollide>
       <material>Gazebo/Orange</material>
-    </gazebo>
+    </gazebo> -->
     <!-- <gazebo reference="virtual_endeffector">
       <selfCollide>false</selfCollide>

File: docker/cyton_ros2/src/ros2_RobotSimulation/Cyton/cyton_ros2_gazebo/urdf/cyton_macros.urdf.xacro (robot description, xacro)
@@ -63,5 +63,5 @@
         </link>
         <!-- First motor located here -->
-        <joint name="shoulder_roll_joint" type="revolute">
+        <joint name="joint1" type="revolute">
             <parent link="base_link" />
             <child link="shoulder_roll" />
@@ -94,5 +94,5 @@
         </link>
         <!-- Second motor located here -->
-        <joint name="shoulder_pitch_joint" type="revolute">
+        <joint name="joint2" type="revolute">
             <parent link="shoulder_roll" />
             <child link="shoulder_pitch" />
@@ -124,7 +124,6 @@
             </inertial>
         </link>
-        <!-- TUTAJ ODPIERDALA -->
         <!-- Third motor located here -->
-        <joint name="elbow_roll_joint" type="revolute">
+        <joint name="joint3" type="revolute">
             <parent link="shoulder_pitch" />
             <child link="elbow_roll" />
@@ -157,5 +156,5 @@
         </link>
         <!-- Fourth motor located here -->
-        <joint name="elbow_pitch_joint" type="revolute">
+        <joint name="joint4" type="revolute">
             <parent link="elbow_roll" />
             <child link="elbow_pitch" />
@@ -189,5 +188,5 @@
         </link>
         <!-- Fifth motor located here -->
-        <joint name="elbow_yaw_joint" type="revolute">
+        <joint name="joint5" type="revolute">
             <parent link="elbow_pitch" />
             <child link="elbow_yaw" />
@@ -220,5 +219,5 @@
         </link>
         <!-- Sixth motor located here -->
-        <joint name="wrist_pitch_joint" type="revolute">
+        <joint name="joint6" type="revolute">
             <parent link="elbow_yaw" />
             <child link="wrist_pitch" />
@@ -251,5 +250,5 @@
         </link>
         <!-- Seventh motor located here -->
-        <joint name="wrist_roll_joint" type="revolute">
+        <joint name="joint7" type="revolute">
             <parent link="wrist_pitch" />
             <child link="wrist_roll" />
@@ -282,5 +281,5 @@
         </link>
         <!-- Eighth motor located here -->
-        <joint name="gripper_joint" type="prismatic">
+        <!-- <joint name="gripper_joint" type="prismatic">
             <parent link="wrist_roll" />
             <child link="gripper_finger1" />
@@ -310,7 +309,7 @@
                     iyy="9.527084112726167e-05" iyz="0" izz="5.193749979697169e-05" />
             </inertial>
-        </link>
+        </link> -->
         <!-- Eighth motor located here -->
-        <joint name="mimic_gripper_joint" type="prismatic">
+        <!-- <joint name="mimic_gripper_joint" type="prismatic">
             <parent link="wrist_roll" />
             <child link="gripper_finger2" />
@@ -341,5 +340,5 @@
                     iyy="9.527084112726167e-05" iyz="0" izz="5.193749979697169e-05" />
             </inertial>
-        </link>
+        </link> -->
         <!-- <xacro:if value="${virtual_ee}">
             <joint name="virtual_endeffector_joint" type="fixed">

File: docker/cyton_ros2/src/ros2_RobotSimulation/Cyton/cyton_ros2_gazebo/urdf/cyton_transmission.xacro (robot description, xacro)
@@ -59,5 +59,5 @@
   <transmission name="tran1">
     <type>transmission_interface/SimpleTransmission</type>
-    <joint name="shoulder_roll_joint">
+    <joint name="joint1">
       <hardwareInterface>PositionJointInterface</hardwareInterface>
     </joint>
@@ -68,5 +68,5 @@
   <transmission name="tran2">
     <type>transmission_interface/SimpleTransmission</type>
-    <joint name="shoulder_pitch_joint">
+    <joint name="joint2">
       <hardwareInterface>PositionJointInterface</hardwareInterface>
     </joint>
@@ -77,5 +77,5 @@
   <transmission name="tran3">
     <type>transmission_interface/SimpleTransmission</type>
-    <joint name="elbow_roll_joint">
+    <joint name="joint3">
       <hardwareInterface>PositionJointInterface</hardwareInterface>
     </joint>
@@ -86,5 +86,5 @@
   <transmission name="tran4">
     <type>transmission_interface/SimpleTransmission</type>
-    <joint name="elbow_pitch_joint">
+    <joint name="joint4">
       <hardwareInterface>PositionJointInterface</hardwareInterface>
     </joint>
@@ -95,5 +95,5 @@
   <transmission name="tran5">
     <type>transmission_interface/SimpleTransmission</type>
-    <joint name="elbow_yaw_joint">
+    <joint name="joint5">
       <hardwareInterface>PositionJointInterface</hardwareInterface>
     </joint>
@@ -104,5 +104,5 @@
   <transmission name="tran6">
     <type>transmission_interface/SimpleTransmission</type>
-    <joint name="wrist_pitch_joint">
+    <joint name="joint6">
       <hardwareInterface>PositionJointInterface</hardwareInterface>
     </joint>
@@ -113,5 +113,5 @@
   <transmission name="tran7">
     <type>transmission_interface/SimpleTransmission</type>
-    <joint name="wrist_roll_joint">
+    <joint name="joint7">
       <hardwareInterface>PositionJointInterface</hardwareInterface>
     </joint>
@@ -120,5 +120,5 @@
     </actuator>
   </transmission>
-  <transmission name="tran8">
+  <!-- <transmission name="tran8">
     <type>transmission_interface/SimpleTransmission</type>
     <joint name="gripper_joint">
@@ -128,5 +128,5 @@
       <hardwareInterface>PositionJointInterface</hardwareInterface>
     </actuator>
-  </transmission>
+  </transmission> -->
 <!-- TODO Motor 9 in reality is motor 8, don't know solution yet -->
   <!-- <transmission name="tran9">
