Commit message: dummy cyton functional (no gripper)

File: docker/cyton_ros2/src/ros2_RobotSimulation/Cyton/cyton_moveit/config/cyton.ros2_control.xacro (robot description, xacro)
@@ -7,5 +7,5 @@
               <plugin>dynamixel_hardware/DynamixelHardware</plugin>
               <param name="usb_port">/dev/ttyUSB0</param>
-              <param name="baud_rate">1000000</param>
+              <param name="baud_rate">57600</param>
               <param name="use_dummy">true</param>
             </hardware>
@@ -24,5 +24,5 @@
                 <command_interface name="position"/>
                 <state_interface name="position">
-                  <param name="initial_value">${initial_positions['shoulder_pitch_joint']}</param>
+                  <param name="initial_value">${initial_positions['joint2']}</param>
                 </state_interface>
                 <state_interface name="velocity"/>
@@ -33,5 +33,5 @@
                 <command_interface name="position"/>
                 <state_interface name="position">
-                  <param name="initial_value">${initial_positions['elbow_roll_joint']}</param>
+                  <param name="initial_value">${initial_positions['joint3']}</param>
                 </state_interface>
                 <state_interface name="velocity"/>
@@ -42,5 +42,5 @@
                 <command_interface name="position"/>
                 <state_interface name="position">
-                  <param name="initial_value">${initial_positions['elbow_pitch_joint']}</param>
+                  <param name="initial_value">${initial_positions['joint4']}</param>
                 </state_interface>
                 <state_interface name="velocity"/>
@@ -51,23 +51,23 @@
                 <command_interface name="position"/>
                 <state_interface name="position">
-                  <param name="initial_value">${initial_positions['elbow_yaw_joint']}</param>
+                  <param name="initial_value">${initial_positions['joint5']}</param>
                 </state_interface>
                 <state_interface name="velocity"/>
             </joint>
             <!-- <joint name="wrist_pitch_joint"> -->
+            <joint name="joint7">
+                <param name="id">7</param>
+                <command_interface name="position"/>
+                <state_interface name="position">
+                  <param name="initial_value">${initial_positions['joint6']}</param>
+                </state_interface>
+                <state_interface name="velocity"/>
+            </joint>
+            <!-- <joint name="wrist_roll_joint"> -->
             <joint name="joint6">
                 <param name="id">6</param>
                 <command_interface name="position"/>
                 <state_interface name="position">
-                  <param name="initial_value">${initial_positions['wrist_pitch_joint']}</param>
-                </state_interface>
-                <state_interface name="velocity"/>
-            </joint>
-            <!-- <joint name="wrist_roll_joint"> -->
-            <joint name="joint7">
-                <param name="id">7</param>
-                <command_interface name="position"/>
-                <state_interface name="position">
-                  <param name="initial_value">${initial_positions['wrist_roll_joint']}</param>
+                  <param name="initial_value">${initial_positions['joint7']}</param>
                 </state_interface>
                 <state_interface name="velocity"/>

File: docker/cyton_ros2/src/ros2_RobotSimulation/Cyton/cyton_ros2_gazebo/urdf/cyton_macros.urdf.xacro (robot description, xacro)
@@ -65,15 +65,15 @@
         <joint name="joint1" type="revolute">
             <parent link="base_link" />
-            <child link="shoulder_roll" />
-            <origin xyz="0 0 0.05315" rpy="0 0 1.2" />
+            <child link="joint1" />
+            <origin xyz="0 0 0.05315" rpy="0 0 0" />
             <dynamics damping="0.5" friction="0.5"/>
             <limit lower="-2.618" upper="2.618" effort="7.0" velocity="1.0" />
             <axis xyz="0 0 1" />
         </joint>
-        <link name="shoulder_roll">
+        <link name="joint1">
             <visual>
                 <origin xyz="0 0 0" rpy="1.5708 0 3.14159" />
                 <geometry>
-                    <mesh filename="file://$(find cyton_ros2_gazebo)/meshes/visual/Shoulder_Roll.dae" />
+                    <mesh filename="file://$(find cyton_ros2_gazebo)/meshes/visual/joint1.dae" />
                 </geometry>
                 <material name="blue"/>
@@ -82,5 +82,5 @@
                 <origin xyz="0 0 0" rpy="1.5708 0 3.14159" />
                 <geometry>
-                    <mesh filename="file://$(find cyton_ros2_gazebo)/meshes/collision/Shoulder_Roll.stl" />
+                    <mesh filename="file://$(find cyton_ros2_gazebo)/meshes/collision/joint1.stl" />
                     <!-- <sphere radius="0.001" /> -->
                 </geometry>
@@ -95,16 +95,16 @@
         <!-- Second motor located here -->
         <joint name="joint2" type="revolute">
-            <parent link="shoulder_roll" />
-            <child link="shoulder_pitch" />
-            <origin xyz="0 0 0.063" rpy="1.2 0 0" />
-            <dynamics damping="0.5" friction="0.5"/>
-            <limit lower="-1.8326" upper="1.8326" effort="7.0" velocity="1.0" />
-            <axis xyz="1 0 0" />
-        </joint>
-        <link name="shoulder_pitch">
+            <parent link="joint1" />
+            <child link="joint2" />
+            <origin xyz="0 0 0.063" rpy="0 0 0" />
+            <dynamics damping="0.5" friction="0.5"/>
+            <limit lower="-1.8326" upper="1.8326" effort="7.0" velocity="1.0" />
+            <axis xyz="1 0 0" />
+        </joint>
+        <link name="joint2">
             <visual>
                 <origin xyz="0.028 0 0" rpy="0 1.5708 0" />
                 <geometry>
-                    <mesh filename="file://$(find cyton_ros2_gazebo)/meshes/visual/Shoulder_Pitch.dae" />
+                    <mesh filename="file://$(find cyton_ros2_gazebo)/meshes/visual/joint2.dae" />
                 </geometry>
                 <material name="blue"/>
@@ -113,5 +113,5 @@
                 <origin xyz="0.028 0 0" rpy="0 1.5708 0" />
                 <geometry>
-                    <mesh filename="file://$(find cyton_ros2_gazebo)/meshes/collision/Shoulder_Pitch.stl" />
+                    <mesh filename="file://$(find cyton_ros2_gazebo)/meshes/collision/joint2.stl" />
                     <!-- <sphere radius="0.001" /> -->
                 </geometry>
@@ -126,16 +126,16 @@
         <!-- Third motor located here -->
         <joint name="joint3" type="revolute">
-            <parent link="shoulder_pitch" />
-            <child link="elbow_roll" />
-            <origin xyz="0 0 0.089" rpy="0 0 1.2" />
+            <parent link="joint2" />
+            <child link="joint3" />
+            <origin xyz="0 0 0.089" rpy="0 0 0" />
             <dynamics damping="0.5" friction="0.5"/>
             <limit lower="-1.8326" upper="1.8326" effort="7.0" velocity="1.0" />
             <axis xyz="0 0 1" />
         </joint>
-        <link name="elbow_roll">
+        <link name="joint3">
             <visual>
                 <origin xyz="0 0 0" rpy="0 0 3.92699" />
                 <geometry>
-                    <mesh filename="file://$(find cyton_ros2_gazebo)/meshes/visual/Elbow_Roll.dae" />
+                    <mesh filename="file://$(find cyton_ros2_gazebo)/meshes/visual/joint3.dae" />
                 </geometry>
                 <material name="blue"/>
@@ -144,5 +144,5 @@
                 <origin xyz="0 0 0" rpy="0 0 3.92699" />
                 <geometry>
-                    <mesh filename="file://$(find cyton_ros2_gazebo)/meshes/collision/Elbow_Roll.stl" />
+                    <mesh filename="file://$(find cyton_ros2_gazebo)/meshes/collision/joint3.stl" />
                     <!-- <sphere radius="0.001" /> -->
                 </geometry>
@@ -157,17 +157,17 @@
         <!-- Fourth motor located here -->
         <joint name="joint4" type="revolute">
-            <parent link="elbow_roll" />
-            <child link="elbow_pitch" />
-            <origin xyz="0 0 0.052" rpy="1.2 0 0" />
-            <dynamics damping="0.5" friction="0.5"/>
-            <limit lower="-1.8326" upper="1.8326" effort="7.0" velocity="1.0" />
-            <axis xyz="1 0 0" />
-        </joint>
-        <link name="elbow_pitch">
+            <parent link="joint3" />
+            <child link="joint4" />
+            <origin xyz="0 0 0.052" rpy="0 0 0" />
+            <dynamics damping="0.5" friction="0.5"/>
+            <limit lower="-1.8326" upper="1.8326" effort="7.0" velocity="1.0" />
+            <axis xyz="1 0 0" />
+        </joint>
+        <link name="joint4">
             <visual>
                 <!-- Not sure if this is the correct orientation. -->
                 <origin xyz="0.027 0 0" rpy="1.5708 0 1.5708" />
                 <geometry>
-                    <mesh filename="file://$(find cyton_ros2_gazebo)/meshes/visual/Elbow_Pitch.dae" />
+                    <mesh filename="file://$(find cyton_ros2_gazebo)/meshes/visual/joint4.dae" />
                 </geometry>
                 <material name="blue"/>
@@ -176,5 +176,5 @@
                 <origin xyz="0.027 0 0" rpy="1.5708 0 1.5708" />
                 <geometry>
-                    <mesh filename="file://$(find cyton_ros2_gazebo)/meshes/collision/Elbow_Pitch.stl" />
+                    <mesh filename="file://$(find cyton_ros2_gazebo)/meshes/collision/joint4.stl" />
                     <!-- <sphere radius="0.001" /> -->
                 </geometry>
@@ -189,16 +189,16 @@
         <!-- Fifth motor located here -->
         <joint name="joint5" type="revolute">
-            <parent link="elbow_pitch" />
-            <child link="elbow_yaw" />
-            <origin xyz="0 0 0.072" rpy="0 -1.2 0" />
+            <parent link="joint4" />
+            <child link="joint5" />
+            <origin xyz="0 0 0.072" rpy="0 0 0" />
             <dynamics damping="0.5" friction="0.5"/>
             <limit lower="-1.8326" upper="1.8326" effort="7.0" velocity="1.0" />
             <axis xyz="0 -1 0" />
         </joint>
-        <link name="elbow_yaw">
+        <link name="joint5">
             <visual>
                 <origin xyz="0 0 0" rpy="1.5708 0 0" />
                 <geometry>
-                    <mesh filename="file://$(find cyton_ros2_gazebo)/meshes/visual/Elbow_Yaw.dae" />
+                    <mesh filename="file://$(find cyton_ros2_gazebo)/meshes/visual/joint5.dae" />
                 </geometry>
                 <material name="blue"/>
@@ -207,5 +207,5 @@
                 <origin xyz="0 0 0" rpy="1.5708 0 0" />
                 <geometry>
-                    <mesh filename="file://$(find cyton_ros2_gazebo)/meshes/collision/Elbow_Yaw.stl" />
+                    <mesh filename="file://$(find cyton_ros2_gazebo)/meshes/collision/joint5.stl" />
                     <!-- <sphere radius="0.001" /> -->
                 </geometry>
@@ -219,17 +219,17 @@
         </link>
         <!-- Sixth motor located here -->
-        <joint name="joint6" type="revolute">
-            <parent link="elbow_yaw" />
-            <child link="wrist_pitch" />
-            <origin xyz="0 0 0.0718" rpy="1.2 0 0" />
-            <dynamics damping="0.5" friction="0.5"/>
-            <limit lower="-1.8326" upper="1.8326" effort="7.0" velocity="1.0" />
-            <axis xyz="1 0 0" />
-        </joint>
-        <link name="wrist_pitch">
+        <joint name="joint7" type="revolute">
+            <parent link="joint5" />
+            <child link="joint7" />
+            <origin xyz="0 0 0.0718" rpy="0 0 0" />
+            <dynamics damping="0.5" friction="0.5"/>
+            <limit lower="-1.8326" upper="1.8326" effort="7.0" velocity="1.0" />
+            <axis xyz="1 0 0" />
+        </joint>
+        <link name="joint7">
             <visual>
                 <origin xyz="0.027 0 0" rpy="1.5708 0 1.5708" />
                 <geometry>
-                    <mesh filename="file://$(find cyton_ros2_gazebo)/meshes/visual/Wrist_Pitch.dae" />
+                    <mesh filename="file://$(find cyton_ros2_gazebo)/meshes/visual/joint7.dae" />
                 </geometry>
                 <material name="blue"/>
@@ -238,5 +238,5 @@
                 <origin xyz="0.027 0 0" rpy="1.5708 0 1.5708" />
                 <geometry>
-                    <mesh filename="file://$(find cyton_ros2_gazebo)/meshes/collision/Wrist_Pitch.stl" />
+                    <mesh filename="file://$(find cyton_ros2_gazebo)/meshes/collision/joint7.stl" />
                     <!-- <sphere radius="0.001" /> -->
                 </geometry>
@@ -250,17 +250,17 @@
         </link>
         <!-- Seventh motor located here -->
-        <joint name="joint7" type="revolute">
-            <parent link="wrist_pitch" />
-            <child link="wrist_roll" />
-            <origin xyz="0 0 0.051425" rpy="0 0 1.2" />
+        <joint name="joint6" type="revolute">
+            <parent link="joint7" />
+            <child link="joint6" />
+            <origin xyz="0 0 0.051425" rpy="0 0 0" />
             <dynamics damping="0.5" friction="0.5"/>
             <limit lower="-2.61799" upper="2.61799" effort="7.0" velocity="1.0" />
             <axis xyz="0 0 1" />
         </joint>
-        <link name="wrist_roll">
+        <link name="joint6">
             <visual>
                 <origin xyz="0 0 0" rpy="0 3.14159 1.5708" />
                 <geometry>
-                    <mesh filename="file://$(find cyton_ros2_gazebo)/meshes/visual/Wrist_Roll.dae" />
+                    <mesh filename="file://$(find cyton_ros2_gazebo)/meshes/visual/joint6.dae" />
                 </geometry>
                 <material name="blue"/>
@@ -269,5 +269,5 @@
                 <origin xyz="0 0 0" rpy="0 3.14159 1.5708" />
                 <geometry>
-                    <mesh filename="file://$(find cyton_ros2_gazebo)/meshes/collision/Wrist_Roll.stl" />
+                    <mesh filename="file://$(find cyton_ros2_gazebo)/meshes/collision/joint6.stl" />
                     <!-- <sphere radius="0.001" /> -->
                 </geometry>
@@ -282,5 +282,5 @@
         <!-- Eighth motor located here -->
         <!-- <joint name="gripper_joint" type="prismatic">
-            <parent link="wrist_roll" />
+            <parent link="joint7" />
             <child link="gripper_finger1" />
             <origin xyz="-0.01331 0.00485 0.077225" rpy="0 0 0" />
@@ -312,5 +312,5 @@
         <!-- Eighth motor located here -->
         <!-- <joint name="mimic_gripper_joint" type="prismatic">
-            <parent link="wrist_roll" />
+            <parent link="joint7" />
             <child link="gripper_finger2" />
             <origin xyz="0.0098 0.00485 0.077225" rpy="0 0 0" />
@@ -343,5 +343,5 @@
         <!-- <xacro:if value="${virtual_ee}">
             <joint name="virtual_endeffector_joint" type="fixed">
-                <parent link="wrist_roll" />
+                <parent link="joint7" />
                 <child link="virtual_endeffector" />
                 <origin xyz="-0.002316 0.0079 0.079425" rpy="0 0 0" />

Commit message: Arm functional (without gripper)

File: docker/cyton_ros2/src/ros2_RobotSimulation/Cyton/cyton_moveit/config/cyton.ros2_control.xacro (robot description, xacro)
@@ -8,5 +8,5 @@
               <param name="usb_port">/dev/ttyUSB0</param>
               <param name="baud_rate">57600</param>
-              <param name="use_dummy">true</param>
+              <!-- <param name="use_dummy">true</param> -->
             </hardware>
             <!-- <joint name="shoulder_roll_joint"> -->
@@ -55,7 +55,7 @@
                 <state_interface name="velocity"/>
             </joint>
-            <!-- <joint name="wrist_pitch_joint"> -->
-            <joint name="joint7">
-                <param name="id">7</param>
+            <!-- <joint name="wrist_roll_joint"> -->
+            <joint name="joint6">
+                <param name="id">6</param>
                 <command_interface name="position"/>
                 <state_interface name="position">
@@ -64,7 +64,7 @@
                 <state_interface name="velocity"/>
             </joint>
-            <!-- <joint name="wrist_roll_joint"> -->
-            <joint name="joint6">
-                <param name="id">6</param>
+            <!-- <joint name="wrist_pitch_joint"> -->
+            <joint name="joint7">
+                <param name="id">7</param>
                 <command_interface name="position"/>
                 <state_interface name="position">

File: docker/cyton_ros2/src/ros2_RobotSimulation/Cyton/cyton_ros2_gazebo/urdf/cyton_ignition.xacro (robot description, xacro)
@@ -143,5 +143,5 @@
       <!-- cyton_joint6 -->
       <!-- <joint name="wrist_pitch_joint"> -->
-      <joint name="joint6">
+      <joint name="joint7">
         <!-- <param name="initial_position">1.5708</param> -->
         <command_interface name="position">
@@ -159,5 +159,5 @@
       <!-- cyton_joint7 -->
       <!-- <joint name="wrist_roll_joint"> -->
-      <joint name="joint7">
+      <joint name="joint6">
         <!-- <param name="initial_position">0.785</param> -->
         <command_interface name="position">

File: docker/cyton_ros2/src/ros2_RobotSimulation/Cyton/cyton_ros2_gazebo/urdf/cyton_macros.urdf.xacro (robot description, xacro)
@@ -219,7 +219,7 @@
         </link>
         <!-- Sixth motor located here -->
-        <joint name="joint7" type="revolute">
+        <joint name="joint6" type="revolute">
             <parent link="joint5" />
-            <child link="joint7" />
+            <child link="joint6" />
             <origin xyz="0 0 0.0718" rpy="0 0 0" />
             <dynamics damping="0.5" friction="0.5"/>
@@ -227,9 +227,9 @@
             <axis xyz="1 0 0" />
         </joint>
-        <link name="joint7">
+        <link name="joint6">
             <visual>
                 <origin xyz="0.027 0 0" rpy="1.5708 0 1.5708" />
                 <geometry>
-                    <mesh filename="file://$(find cyton_ros2_gazebo)/meshes/visual/joint7.dae" />
+                    <mesh filename="file://$(find cyton_ros2_gazebo)/meshes/visual/joint6.dae" />
                 </geometry>
                 <material name="blue"/>
@@ -238,5 +238,5 @@
                 <origin xyz="0.027 0 0" rpy="1.5708 0 1.5708" />
                 <geometry>
-                    <mesh filename="file://$(find cyton_ros2_gazebo)/meshes/collision/joint7.stl" />
+                    <mesh filename="file://$(find cyton_ros2_gazebo)/meshes/collision/joint6.stl" />
                     <!-- <sphere radius="0.001" /> -->
                 </geometry>
@@ -250,17 +250,17 @@
         </link>
         <!-- Seventh motor located here -->
-        <joint name="joint6" type="revolute">
-            <parent link="joint7" />
-            <child link="joint6" />
-            <origin xyz="0 0 0.051425" rpy="0 0 0" />
+        <joint name="joint7" type="revolute">
+            <parent link="joint6" />
+            <child link="joint7" />
+            <origin xyz="0 0 0.051425" rpy="0 0 3.1416" />
             <dynamics damping="0.5" friction="0.5"/>
             <limit lower="-2.61799" upper="2.61799" effort="7.0" velocity="1.0" />
             <axis xyz="0 0 1" />
         </joint>
-        <link name="joint6">
+        <link name="joint7">
             <visual>
                 <origin xyz="0 0 0" rpy="0 3.14159 1.5708" />
                 <geometry>
-                    <mesh filename="file://$(find cyton_ros2_gazebo)/meshes/visual/joint6.dae" />
+                    <mesh filename="file://$(find cyton_ros2_gazebo)/meshes/visual/joint7.dae" />
                 </geometry>
                 <material name="blue"/>
@@ -269,5 +269,5 @@
                 <origin xyz="0 0 0" rpy="0 3.14159 1.5708" />
                 <geometry>
-                    <mesh filename="file://$(find cyton_ros2_gazebo)/meshes/collision/joint6.stl" />
+                    <mesh filename="file://$(find cyton_ros2_gazebo)/meshes/collision/joint7.stl" />
                     <!-- <sphere radius="0.001" /> -->
                 </geometry>
