Commit message: gripper problem

File: docker/cyton_ros2/src/ros2_RobotSimulation/Cyton/cyton_moveit/config/cyton.ros2_control.xacro (robot description, xacro)
@@ -8,5 +8,5 @@
               <param name="usb_port">/dev/ttyUSB0</param>
               <param name="baud_rate">115200</param>
-              <param name="use_dummy">true</param>
+              <!-- <param name="use_dummy">true</param> -->
             </hardware>
             <joint name="joint1">

File: docker/cyton_ros2/src/ros2_RobotSimulation/Cyton/cyton_ros2_gazebo/urdf/cyton_macros.urdf.xacro (robot description, xacro)
@@ -218,8 +218,39 @@
             </inertial>
         </link>
+        <!-- Seventh motor located here -->
+        <joint name="joint7" type="revolute">
+            <parent link="joint6" />
+            <child link="joint7" />
+            <origin xyz="0 0 0.051425" rpy="0 0 0" />
+            <dynamics damping="0.5" friction="0.5"/>
+            <limit lower="-2.61799" upper="2.61799" effort="7.0" velocity="1.0" />
+            <axis xyz="0 0 1" />
+        </joint>
+        <link name="joint7">
+            <visual>
+                <origin xyz="0 0 0" rpy="0 3.14159 1.5708" />
+                <geometry>
+                    <mesh filename="file://$(find cyton_ros2_gazebo)/meshes/visual/joint6.dae" />
+                </geometry>
+                <material name="blue"/>
+            </visual>
+            <collision>
+                <origin xyz="0 0 0" rpy="0 3.14159 1.5708" />
+                <geometry>
+                    <mesh filename="file://$(find cyton_ros2_gazebo)/meshes/collision/joint6.stl" />
+                    <!-- <sphere radius="0.001" /> -->
+                </geometry>
+            </collision>
+            <inertial>
+                <mass value="1.0" />
+                <origin rpy="0 0 0" xyz="0 0 0" />
+                <inertia  ixx="0.0015572863522148085" ixy="0" ixz="0"
+                    iyy="0.0015598712477069795" iyz="0" izz="0.002615797579411179" />
+            </inertial>
+        </link>
         <!-- Sixth motor located here -->
-        <joint name="joint7" type="revolute">
+        <joint name="joint6" type="revolute">
             <parent link="joint5" />
-            <child link="joint7" />
+            <child link="joint6" />
             <origin xyz="0 0 0.0718" rpy="0 0 0" />
             <dynamics damping="0.5" friction="0.5"/>
@@ -227,5 +258,5 @@
             <axis xyz="1 0 0" />
         </joint>
-        <link name="joint7">
+        <link name="joint6">
             <visual>
                 <origin xyz="0.027 0 0" rpy="1.5708 0 1.5708" />
@@ -249,38 +280,7 @@
             </inertial>
         </link>
-        <!-- Seventh motor located here -->
-        <joint name="joint6" type="revolute">
-            <parent link="joint7" />
-            <child link="joint6" />
-            <origin xyz="0 0 0.051425" rpy="0 0 0" />
-            <dynamics damping="0.5" friction="0.5"/>
-            <limit lower="-2.61799" upper="2.61799" effort="7.0" velocity="1.0" />
-            <axis xyz="0 0 1" />
-        </joint>
-        <link name="joint6">
-            <visual>
-                <origin xyz="0 0 0" rpy="0 3.14159 1.5708" />
-                <geometry>
-                    <mesh filename="file://$(find cyton_ros2_gazebo)/meshes/visual/joint6.dae" />
-                </geometry>
-                <material name="blue"/>
-            </visual>
-            <collision>
-                <origin xyz="0 0 0" rpy="0 3.14159 1.5708" />
-                <geometry>
-                    <mesh filename="file://$(find cyton_ros2_gazebo)/meshes/collision/joint6.stl" />
-                    <!-- <sphere radius="0.001" /> -->
-                </geometry>
-            </collision>
-            <inertial>
-                <mass value="1.0" />
-                <origin rpy="0 0 0" xyz="0 0 0" />
-                <inertia  ixx="0.0015572863522148085" ixy="0" ixz="0"
-                    iyy="0.0015598712477069795" iyz="0" izz="0.002615797579411179" />
-            </inertial>
-        </link>
         <!-- Eighth motor located here -->
         <joint name="joint8" type="prismatic">
-            <parent link="joint6" />
+            <parent link="joint7" />
             <child link="joint8" />
             <origin xyz="-0.01331 0.00485 0.077225" rpy="0 0 0" />
@@ -312,5 +312,5 @@
         <!-- Eighth motor located here -->
         <joint name="joint9" type="prismatic">
-            <parent link="joint6" />
+            <parent link="joint7" />
             <child link="joint9" />
             <origin xyz="0.0098 0.00485 0.077225" rpy="0 0 0" />

Commit message: urdf fixed

File: docker/cyton_ros2/src/ros2_RobotSimulation/Cyton/cyton_moveit/config/cyton.ros2_control.xacro (robot description, xacro)
@@ -5,8 +5,9 @@
         <ros2_control name="${name}" type="system">
             <hardware>
-              <plugin>dynamixel_hardware/DynamixelHardware</plugin>
-              <param name="usb_port">/dev/ttyUSB0</param>
-              <param name="baud_rate">115200</param>
+              <!-- <plugin>dynamixel_hardware/DynamixelHardware</plugin> -->
+              <!-- <param name="usb_port">/dev/ttyUSB0</param> -->
+              <!-- <param name="baud_rate">115200</param> -->
               <!-- <param name="use_dummy">true</param> -->
+              <plugin>mock_components/GenericSystem</plugin>
             </hardware>
             <joint name="joint1">

File: docker/cyton_ros2/src/ros2_RobotSimulation/Cyton/cyton_ros2_gazebo/urdf/cyton_macros.urdf.xacro (robot description, xacro)
@@ -218,4 +218,35 @@
             </inertial>
         </link>
+        <!-- Sixth motor located here -->
+        <joint name="joint6" type="revolute">
+            <parent link="joint5" />
+            <child link="joint6" />
+            <origin xyz="0 0 0.0718" rpy="0 0 0" />
+            <dynamics damping="0.5" friction="0.5"/>
+            <limit lower="-1.8326" upper="1.8326" effort="7.0" velocity="1.0" />
+            <axis xyz="1 0 0" />
+        </joint>
+        <link name="joint6">
+            <visual>
+                <origin xyz="0.027 0 0" rpy="1.5708 0 1.5708" />
+                <geometry>
+                    <mesh filename="file://$(find cyton_ros2_gazebo)/meshes/visual/joint6.dae" />
+                </geometry>
+                <material name="blue"/>
+            </visual>
+            <collision>
+                <origin xyz="0.027 0 0" rpy="1.5708 0 1.5708" />
+                <geometry>
+                    <mesh filename="file://$(find cyton_ros2_gazebo)/meshes/collision/joint6.stl" />
+                    <!-- <sphere radius="0.001" /> -->
+                </geometry>
+            </collision>
+            <inertial>
+                <mass value="1.0" />
+                <origin rpy="0 0 0" xyz="0 0 0" />
+                <inertia  ixx="0.002306163215052582" ixy="0" ixz="0"
+                    iyy="0.003544626555053466" iyz="0" izz="0.004174319112083028" />
+            </inertial>
+        </link>
         <!-- Seventh motor located here -->
         <joint name="joint7" type="revolute">
@@ -231,5 +262,5 @@
                 <origin xyz="0 0 0" rpy="0 3.14159 1.5708" />
                 <geometry>
-                    <mesh filename="file://$(find cyton_ros2_gazebo)/meshes/visual/joint6.dae" />
+                    <mesh filename="file://$(find cyton_ros2_gazebo)/meshes/visual/joint7.dae" />
                 </geometry>
                 <material name="blue"/>
@@ -238,5 +269,5 @@
                 <origin xyz="0 0 0" rpy="0 3.14159 1.5708" />
                 <geometry>
-                    <mesh filename="file://$(find cyton_ros2_gazebo)/meshes/collision/joint6.stl" />
+                    <mesh filename="file://$(find cyton_ros2_gazebo)/meshes/collision/joint7.stl" />
                     <!-- <sphere radius="0.001" /> -->
                 </geometry>
@@ -247,35 +278,4 @@
                 <inertia  ixx="0.0015572863522148085" ixy="0" ixz="0"
                     iyy="0.0015598712477069795" iyz="0" izz="0.002615797579411179" />
-            </inertial>
-        </link>
-        <!-- Sixth motor located here -->
-        <joint name="joint6" type="revolute">
-            <parent link="joint5" />
-            <child link="joint6" />
-            <origin xyz="0 0 0.0718" rpy="0 0 0" />
-            <dynamics damping="0.5" friction="0.5"/>
-            <limit lower="-1.8326" upper="1.8326" effort="7.0" velocity="1.0" />
-            <axis xyz="1 0 0" />
-        </joint>
-        <link name="joint6">
-            <visual>
-                <origin xyz="0.027 0 0" rpy="1.5708 0 1.5708" />
-                <geometry>
-                    <mesh filename="file://$(find cyton_ros2_gazebo)/meshes/visual/joint7.dae" />
-                </geometry>
-                <material name="blue"/>
-            </visual>
-            <collision>
-                <origin xyz="0.027 0 0" rpy="1.5708 0 1.5708" />
-                <geometry>
-                    <mesh filename="file://$(find cyton_ros2_gazebo)/meshes/collision/joint7.stl" />
-                    <!-- <sphere radius="0.001" /> -->
-                </geometry>
-            </collision>
-            <inertial>
-                <mass value="1.0" />
-                <origin rpy="0 0 0" xyz="0 0 0" />
-                <inertia  ixx="0.002306163215052582" ixy="0" ixz="0"
-                    iyy="0.003544626555053466" iyz="0" izz="0.004174319112083028" />
             </inertial>
         </link>

Commit message: everything works, testing

File: docker/cyton_ros2/src/ros2_RobotSimulation/Cyton/cyton_moveit/config/cyton.ros2_control.xacro (robot description, xacro)
@@ -70,5 +70,5 @@
             <joint name="joint8">
                 <param name="id">8</param>
-                <param name="position_multiplier">163.625</param>
+                <param name="position_multiplier">-134.175</param>
                 <command_interface name="position"/>
                 <state_interface name="position">

File: docker/cyton_ros2/src/ros2_RobotSimulation/Cyton/cyton_ros2_gazebo/urdf/cyton_macros.urdf.xacro (robot description, xacro)
@@ -284,9 +284,17 @@
             <parent link="joint7" />
             <child link="joint8" />
-            <origin xyz="-0.01331 0.00485 0.077225" rpy="0 0 0" />
-            <dynamics damping="0.5" friction="0.5"/>
-            <limit lower="-0.008" upper="0.008" effort="7.0" velocity="1.0" />
-            <axis xyz="1 0 0" />
-        </joint>
+            <origin xyz="-0.02131 0.00485 0.077225" rpy="0 0 0" />
+            <dynamics damping="0.5" friction="0.5"/>
+            <limit lower="-0.001" upper="0.017" effort="7.0" velocity="1.0" />
+            <axis xyz="1 0 0" />
+        </joint>
+        <!-- <joint name="joint8" type="prismatic">
+            <parent link="joint7" />
+            <child link="joint8" />
+            <origin xyz="-0.05331 0.00485 0.077225" rpy="0 0 0" />
+            <dynamics damping="0.5" friction="0.5"/>
+            <limit lower="-0.001" upper="0.017" effort="7.0" velocity="1.0" />
+            <axis xyz="1 0 0" />
+        </joint> -->
         <link name="joint8">
             <visual>
@@ -314,10 +322,20 @@
             <parent link="joint7" />
             <child link="joint9" />
-            <origin xyz="0.0098 0.00485 0.077225" rpy="0 0 0" />
-            <dynamics damping="0.5" friction="0.5"/>
-            <limit lower="-0.008" upper="0.008" effort="7.0" velocity="1.0" />
+            <origin xyz="0.0178 0.00485 0.077225" rpy="0 0 0" />
+            <dynamics damping="0.5" friction="0.5"/>
+            <limit lower="-0.017" upper="0.001" effort="7.0" velocity="1.0" />
             <mimic joint="joint8" multiplier="-1"/>
             <axis xyz="1 0 0" />
         </joint>
+<!--
+        <joint name="joint9" type="prismatic">
+            <parent link="joint7" />
+            <child link="joint9" />
+            <origin xyz="0.0498 0.00485 0.077225" rpy="0 0 0" />
+            <dynamics damping="0.5" friction="0.5"/>
+            <limit lower="-0.017" upper="0.001" effort="7.0" velocity="1.0" />
+            <mimic joint="joint8" multiplier="-1"/>
+            <axis xyz="1 0 0" />
+        </joint> -->
         <link name="joint9">
             <visual>
