Commit message: sim works, moveit not

File: docker/cyton_ros2/src/ros2_RobotSimulation/Cyton/cyton_moveit/config/cyton.ros2_control.xacro (robot description, xacro)
@@ -4,12 +4,16 @@
         <xacro:property name="initial_positions" value="${load_yaml(initial_positions_file)['initial_positions']}"/>
         <ros2_control name="${name}" type="system">
-            <hardware>
+            <!-- <hardware>
               <plugin>dynamixel_hardware/DynamixelHardware</plugin>
               <param name="usb_port">/dev/ttyUSB0</param>
               <param name="baud_rate">115200</param>
-              <param name="joint_ids">1,2,3,4,5,6,7,8</param>
+              <param name="joint_ids">1,2,3,4,5,6,7,8</param> -->
               <!-- <param name="use_dummy">true</param> -->
               <!-- <plugin>mock_components/GenericSystem</plugin> -->
-            </hardware>
+            <!-- </hardware> -->
+                  <!-- <xacro:if value="${use_sim}"> -->
+            <hardware>
+                <plugin>ign_ros2_control/IgnitionSystem</plugin>
+              </hardware>
             <joint name="joint1">
                 <param name="id">1</param>

File: docker/cyton_ros2/src/ros2_RobotSimulation/Cyton/cyton_moveit/config/cyton.urdf.xacro (robot description, xacro)
@@ -5,5 +5,5 @@
     <xacro:include filename="$(find cyton_ros2_gazebo)/urdf/cyton.urdf.xacro" />
     <!-- Import control_xacro -->
-    <xacro:include filename="cyton.ros2_control.xacro" />
-    <xacro:cyton_ros2_control name="DynamixelHardware" initial_positions_file="$(arg initial_positions_file)"/>
+    <!-- <xacro:include filename="cyton.ros2_control.xacro" /> -->
+    <!-- <xacro:cyton_ros2_control name="DynamixelHardware" initial_positions_file="$(arg initial_positions_file)"/> -->
 </robot>

File: docker/cyton_ros2/src/ros2_RobotSimulation/Cyton/cyton_ros2_gazebo/urdf/cyton_ignition.xacro (robot description, xacro)
@@ -136,4 +136,19 @@
         <state_interface name="effort"/>
       </joint>
+            <!-- cyton_joint7 -->
+      <joint name="joint6">
+        <!-- <param name="initial_position">0.785</param> -->
+        <command_interface name="position">
+          <param name="min">-3.15</param> <!-- ** -3.935 -->
+          <param name="max">3.15</param> <!-- ** 2.365 -->
+        </command_interface>
+        <command_interface name="velocity">
+          <param name="min">-2.6100</param>
+          <param name="max">2.6100</param>
+        </command_interface>
+        <state_interface name="position"/>
+        <state_interface name="velocity"/>
+        <state_interface name="effort"/>
+      </joint>
       <!-- cyton_joint6 -->
       <joint name="joint7">
@@ -152,5 +167,5 @@
       </joint>
       <!-- cyton_joint7 -->
-      <joint name="joint6">
+      <joint name="joint8">
         <!-- <param name="initial_position">0.785</param> -->
         <command_interface name="position">
@@ -166,40 +181,4 @@
         <state_interface name="effort"/>
       </joint>
-      <!-- cyton_joint7 -->
-      <joint name="joint8">
-        <!-- <param name="initial_position">0.785</param> -->
-        <command_interface name="position">
-          <param name="min">-3.15</param> <!-- ** -3.935 -->
-          <param name="max">3.15</param> <!-- ** 2.365 -->
-        </command_interface>
-        <command_interface name="velocity">
-          <param name="min">-2.6100</param>
-          <param name="max">2.6100</param>
-        </command_interface>
-        <state_interface name="position"/>
-        <state_interface name="velocity"/>
-        <state_interface name="effort"/>
-      </joint>
-      <!-- cyton_joint7 -->
-      <joint name="joint9">
-        <state_interface name="position"/>
-        <state_interface name="velocity"/>
-        <state_interface name="effort"/>
-      </joint>
-      <!-- cyton_finger_joint1 -->
-      <joint name="joint8">
-        <command_interface name="position">
-          <param name="min">-0.001</param>
-          <param name="max">0.04</param>
-        </command_interface>
-        <command_interface name="velocity">
-          <param name="min">-0.3</param>
-          <param name="max">0.3</param>
-        </command_interface>
-        <state_interface name="position"/>
-        <state_interface name="velocity"/>
-        <state_interface name="effort"/>
-      </joint>
-      <!-- cyton_finger_joint2 -->
       <joint name="joint9">
         <state_interface name="position"/>

File: docker/cyton_ros2/src/ros2_RobotSimulation/Cyton/cyton_ros2_gazebo/urdf/cyton_macros.urdf.xacro (robot description, xacro)
@@ -2,8 +2,8 @@
 <robot xmlns:xacro="http://www.ros.org/wiki/xacro">
     <xacro:include filename="$(find cyton_ros2_gazebo)/urdf/cyton_ignition.xacro" />
-    <xacro:include filename="$(find cyton_ros2_gazebo)/urdf/cyton_transmission.xacro" />
+    <!-- <xacro:include filename="$(find cyton_ros2_gazebo)/urdf/cyton_transmission.xacro" /> -->
     <xacro:macro name="cyton_robot">
-        <xacro:cyton_transmission />
-        <!-- <xacro:cyton_ignition /> -->
+        <!-- <xacro:cyton_transmission /> -->
+        <xacro:cyton_ignition />
         <material name="blue">
           <color rgba= "255 149 0 1"/>
@@ -65,11 +65,11 @@
         <joint name="joint1" type="revolute">
             <parent link="base_link" />
-            <child link="joint1" />
+            <child link="link1" />
             <origin xyz="0 0 0.05315" rpy="0 0 0" />
             <dynamics damping="0.5" friction="0.5"/>
-            <limit lower="-2.618" upper="2.618" effort="7.0" velocity="1.0" />
+            <limit lower="-2.618" upper="2.618" effort="1.0" velocity="1.0" />
             <axis xyz="0 0 1" />
         </joint>
-        <link name="joint1">
+        <link name="link1">
             <visual>
                 <origin xyz="0 0 0" rpy="1.5708 0 3.14159" />
@@ -83,5 +83,4 @@
                 <geometry>
                     <mesh filename="file://$(find cyton_ros2_gazebo)/meshes/collision/joint1.stl" />
-                    <!-- <sphere radius="0.001" /> -->
                 </geometry>
             </collision>
@@ -95,12 +94,12 @@
         <!-- Second motor located here -->
         <joint name="joint2" type="revolute">
-            <parent link="joint1" />
-            <child link="joint2" />
+            <parent link="link1" />
+            <child link="link2" />
             <origin xyz="0 0 0.063" rpy="0 0 0" />
             <dynamics damping="0.5" friction="0.5"/>
-            <limit lower="-1.8326" upper="1.8326" effort="7.0" velocity="1.0" />
-            <axis xyz="1 0 0" />
-        </joint>
-        <link name="joint2">
+            <limit lower="-1.8326" upper="1.8326" effort="1.0" velocity="1.0" />
+            <axis xyz="1 0 0" />
+        </joint>
+        <link name="link2">
             <visual>
                 <origin xyz="0.028 0 0" rpy="0 1.5708 0" />
@@ -114,5 +113,4 @@
                 <geometry>
                     <mesh filename="file://$(find cyton_ros2_gazebo)/meshes/collision/joint2.stl" />
-                    <!-- <sphere radius="0.001" /> -->
                 </geometry>
             </collision>
@@ -126,12 +124,13 @@
         <!-- Third motor located here -->
         <joint name="joint3" type="revolute">
-            <parent link="joint2" />
-            <child link="joint3" />
+            <parent link="link2" />
+            <child link="link3" />
             <origin xyz="0 0 0.089" rpy="0 0 0" />
             <dynamics damping="0.5" friction="0.5"/>
-            <limit lower="-1.8326" upper="1.8326" effort="7.0" velocity="1.0" />
+            <limit lower="-1.8326" upper="1.8326" effort="1.0" velocity="1.0" />
             <axis xyz="0 0 1" />
         </joint>
-        <link name="joint3">
++
+        <link name="link3">
             <visual>
                 <origin xyz="0 0 0" rpy="0 0 3.92699" />
@@ -157,12 +156,12 @@
         <!-- Fourth motor located here -->
         <joint name="joint4" type="revolute">
-            <parent link="joint3" />
-            <child link="joint4" />
+            <parent link="link3" />
+            <child link="link4" />
             <origin xyz="0 0 0.052" rpy="0 0 0" />
             <dynamics damping="0.5" friction="0.5"/>
-            <limit lower="-1.8326" upper="1.8326" effort="7.0" velocity="1.0" />
-            <axis xyz="1 0 0" />
-        </joint>
-        <link name="joint4">
+            <limit lower="-1.8326" upper="1.8326" effort="1.0" velocity="1.0" />
+            <axis xyz="1 0 0" />
+        </joint>
+        <link name="link4">
             <visual>
                 <!-- Not sure if this is the correct orientation. -->
@@ -189,12 +188,12 @@
         <!-- Fifth motor located here -->
         <joint name="joint5" type="revolute">
-            <parent link="joint4" />
-            <child link="joint5" />
+            <parent link="link4" />
+            <child link="link5" />
             <origin xyz="0 0 0.072" rpy="0 0 0" />
             <dynamics damping="0.5" friction="0.5"/>
-            <limit lower="-1.8326" upper="1.8326" effort="7.0" velocity="1.0" />
+            <limit lower="-1.8326" upper="1.8326" effort="1.0" velocity="1.0" />
             <axis xyz="0 -1 0" />
         </joint>
-        <link name="joint5">
+        <link name="link5">
             <visual>
                 <origin xyz="0 0 0" rpy="1.5708 0 0" />
@@ -220,12 +219,12 @@
         <!-- Sixth motor located here -->
         <joint name="joint6" type="revolute">
-            <parent link="joint5" />
-            <child link="joint6" />
+            <parent link="link5" />
+            <child link="link6" />
             <origin xyz="0 0 0.0718" rpy="0 0 0" />
             <dynamics damping="0.5" friction="0.5"/>
-            <limit lower="-1.8326" upper="1.8326" effort="7.0" velocity="1.0" />
-            <axis xyz="1 0 0" />
-        </joint>
-        <link name="joint6">
+            <limit lower="-1.8326" upper="1.8326" effort="1.0" velocity="1.0" />
+            <axis xyz="1 0 0" />
+        </joint>
+        <link name="link6">
             <visual>
                 <origin xyz="0.027 0 0" rpy="1.5708 0 1.5708" />
@@ -251,12 +250,12 @@
         <!-- Seventh motor located here -->
         <joint name="joint7" type="revolute">
-            <parent link="joint6" />
-            <child link="joint7" />
-            <origin xyz="0 0 0.051425" rpy="0 0 0" />
-            <dynamics damping="0.5" friction="0.5"/>
-            <limit lower="-2.61799" upper="2.61799" effort="7.0" velocity="1.0" />
+            <parent link="link6" />
+            <child link="link7" />
+            <origin xyz="0 0 0.051425" rpy="0 0 1.5708" />
+            <dynamics damping="0.5" friction="0.5"/>
+            <limit lower="-2.61799" upper="2.61799" effort="1.0" velocity="1.0" />
             <axis xyz="0 0 1" />
         </joint>
-        <link name="joint7">
+        <link name="link7">
             <visual>
                 <origin xyz="0 0 0" rpy="0 3.14159 1.5708" />
@@ -282,9 +281,9 @@
         <!-- Eighth motor located here -->
         <joint name="joint8" type="prismatic">
-            <parent link="joint7" />
-            <child link="joint8" />
+            <parent link="link7" />
+            <child link="link8" />
             <origin xyz="-0.02131 0.00485 0.077225" rpy="0 0 0" />
             <dynamics damping="0.5" friction="0.5"/>
-            <limit lower="-0.001" upper="0.017" effort="7.0" velocity="1.0" />
+            <limit lower="-0.001" upper="0.017" effort="1.0" velocity="1.0" />
             <axis xyz="1 0 0" />
         </joint>
@@ -294,8 +293,8 @@
             <origin xyz="-0.05331 0.00485 0.077225" rpy="0 0 0" />
             <dynamics damping="0.5" friction="0.5"/>
-            <limit lower="-0.001" upper="0.017" effort="7.0" velocity="1.0" />
+            <limit lower="-0.001" upper="0.017" effort="1.0" velocity="1.0" />
             <axis xyz="1 0 0" />
         </joint> -->
-        <link name="joint8">
+        <link name="link8">
             <visual>
                 <origin xyz="0 0 -0.03" rpy="0 0 0" />
@@ -320,9 +319,9 @@
         <!-- Eighth motor located here -->
         <joint name="joint9" type="prismatic">
-            <parent link="joint7" />
-            <child link="joint9" />
+            <parent link="link7" />
+            <child link="link9" />
             <origin xyz="0.0178 0.00485 0.077225" rpy="0 0 0" />
             <dynamics damping="0.5" friction="0.5"/>
-            <limit lower="-0.017" upper="0.001" effort="7.0" velocity="1.0" />
+            <limit lower="-0.017" upper="0.001" effort="1.0" velocity="1.0" />
             <mimic joint="joint8" multiplier="-1"/>
             <axis xyz="1 0 0" />
@@ -334,9 +333,9 @@
             <origin xyz="0.0498 0.00485 0.077225" rpy="0 0 0" />
             <dynamics damping="0.5" friction="0.5"/>
-            <limit lower="-0.017" upper="0.001" effort="7.0" velocity="1.0" />
+            <limit lower="-0.017" upper="0.001" effort="1.0" velocity="1.0" />
             <mimic joint="joint8" multiplier="-1"/>
             <axis xyz="1 0 0" />
         </joint> -->
-        <link name="joint9">
+        <link name="link9">
             <visual>
                 <origin xyz="0 0 -0.03" rpy="0 0 0" />

Commit message: everything works

File: docker/cyton_ros2/src/ros2_RobotSimulation/Cyton/cyton_moveit/config/cyton.ros2_control.xacro (robot description, xacro)
@@ -81,10 +81,4 @@
                 <state_interface name="velocity"/>
             </joint>
-            <!-- <joint name="joint9">
-                <state_interface name="position">
-                  <param name="initial_value">${initial_positions['joint9']}</param>
-                </state_interface>
-                <state_interface name="velocity"/>
-            </joint> -->
         </ros2_control>
     </xacro:macro>

File: docker/cyton_ros2/src/ros2_RobotSimulation/Cyton/cyton_ros2_gazebo/urdf/cyton_ignition.xacro (robot description, xacro)
@@ -183,7 +183,7 @@
       <joint name="joint9">
         <param name="mimic">joint8</param>
-        <state_interface name="position"/>
-        <state_interface name="velocity"/>
-        <state_interface name="effort"/>
+        <param name="multiplier">-1</param>
+        <command_interface name="position"></command_interface>
+        <state_interface name="position"></state_interface>
       </joint>
     </ros2_control>
@@ -220,5 +220,5 @@
       <material>Gazebo/Orange</material>
     </gazebo>
-    <gazebo reference="joint9_mimic">
+    <gazebo reference="joint9">
       <selfCollide>false</selfCollide>
       <material>Gazebo/Orange</material>

File: docker/cyton_ros2/src/ros2_RobotSimulation/Cyton/cyton_ros2_gazebo/urdf/cyton_macros.urdf.xacro (robot description, xacro)
@@ -318,5 +318,5 @@
         </link>
         <!-- Eighth motor located here -->
-        <joint name="joint9_mimic" type="prismatic">
+        <joint name="joint9" type="prismatic">
             <parent link="link7" />
             <child link="link9" />
@@ -327,14 +327,4 @@
             <axis xyz="1 0 0" />
         </joint>
-<!--
-        <joint name="joint9" type="prismatic">
-            <parent link="joint7" />
-            <child link="joint9" />
-            <origin xyz="0.0498 0.00485 0.077225" rpy="0 0 0" />
-            <dynamics damping="0.5" friction="0.5"/>
-            <limit lower="-0.017" upper="0.001" effort="100.0" velocity="1.0" />
-            <mimic joint="joint8" multiplier="-1"/>
-            <axis xyz="1 0 0" />
-        </joint> -->
         <link name="link9">
             <visual>
