Commit message: work in progress

File: src/cyton_bringup/urdf/cyton.hardware.xacro (robot description, xacro)
@@ -1,18 +1,12 @@
 <?xml version="1.0"?>
 <robot xmlns:xacro="http://www.ros.org/wiki/xacro">
-    <xacro:macro name="cyton_ros2_control" params="name initial_positions_file">
-        <xacro:property name="initial_positions" value="${load_yaml(initial_positions_file)['initial_positions']}"/>
-        <ros2_control name="${name}" type="system">
-            <!-- <hardware>
+      <xacro:macro name="cyton_hardware">
+        <!-- <xacro:property name="initial_positions" value="${load_yaml(initial_positions_file)['initial_positions']}"/> -->
+        <ros2_control name="DynamixelHardware" type="system">
+            <hardware>
               <plugin>dynamixel_hardware/DynamixelHardware</plugin>
               <param name="usb_port">/dev/ttyUSB0</param>
               <param name="baud_rate">115200</param>
-              <param name="joint_ids">1,2,3,4,5,6,7,8</param> -->
-              <!-- <param name="use_dummy">true</param> -->
-              <!-- <plugin>mock_components/GenericSystem</plugin> -->
-            <!-- </hardware> -->
-                  <!-- <xacro:if value="${use_sim}"> -->
-            <hardware>
-                <plugin>ign_ros2_control/IgnitionSystem</plugin>
+              <param name="joint_ids">1,2,3,4,5,6,7,8</param>
             </hardware>
             <joint name="joint1">
@@ -20,5 +14,5 @@
                 <command_interface name="position"/>
                 <state_interface name="position">
-                  <param name="initial_value">${initial_positions['joint1']}</param>
+                  <!-- <param name="initial_value">${initial_positions['joint1']}</param> -->
                 </state_interface>
                 <state_interface name="velocity"/>
@@ -28,5 +22,5 @@
                 <command_interface name="position"/>
                 <state_interface name="position">
-                  <param name="initial_value">${initial_positions['joint2']}</param>
+                  <!-- <param name="initial_value">${initial_positions['joint2']}</param> -->
                 </state_interface>
                 <state_interface name="velocity"/>
@@ -36,5 +30,5 @@
                 <command_interface name="position"/>
                 <state_interface name="position">
-                  <param name="initial_value">${initial_positions['joint3']}</param>
+                  <!-- <param name="initial_value">${initial_positions['joint3']}</param> -->
                 </state_interface>
                 <state_interface name="velocity"/>
@@ -44,5 +38,5 @@
                 <command_interface name="position"/>
                 <state_interface name="position">
-                  <param name="initial_value">${initial_positions['joint4']}</param>
+                  <!-- <param name="initial_value">${initial_positions['joint4']}</param> -->
                 </state_interface>
                 <state_interface name="velocity"/>
@@ -52,5 +46,5 @@
                 <command_interface name="position"/>
                 <state_interface name="position">
-                  <param name="initial_value">${initial_positions['joint5']}</param>
+                  <!-- <param name="initial_value">${initial_positions['joint5']}</param> -->
                 </state_interface>
                 <state_interface name="velocity"/>
@@ -60,5 +54,5 @@
                 <command_interface name="position"/>
                 <state_interface name="position">
-                  <param name="initial_value">${initial_positions['joint6']}</param>
+                  <!-- <param name="initial_value">${initial_positions['joint6']}</param> -->
                 </state_interface>
                 <state_interface name="velocity"/>
@@ -68,5 +62,5 @@
                 <command_interface name="position"/>
                 <state_interface name="position">
-                  <param name="initial_value">${initial_positions['joint7']}</param>
+                  <!-- <param name="initial_value">${initial_positions['joint7']}</param> -->
                 </state_interface>
                 <state_interface name="velocity"/>
@@ -77,5 +71,5 @@
                 <command_interface name="position"/>
                 <state_interface name="position">
-                  <param name="initial_value">${initial_positions['joint8']}</param>
+                  <!-- <param name="initial_value">${initial_positions['joint8']}</param> -->
                 </state_interface>
                 <state_interface name="velocity"/>

File: src/cyton_bringup/urdf/cyton_ignition.xacro (robot description, xacro)
@@ -50,10 +50,6 @@
     <gazebo>
       <plugin name="ign_ros2_control::IgnitionROS2ControlPlugin" filename="libign_ros2_control-system.so" >
-      <parameters> $(find cyton_ros2_gazebo)/config/cyton_controller.yaml </parameters>
-      <!-- <controller_manager_node_name>controller_manager</controller_manager_node_name> -->
-      <!-- <robotSimType>gazebo_ros2_control/DefaultRobotHWSim</robotSimType>
-            <robot_param>robot_description</robot_param>
-            <robot_param_node>robot_state_publisher</robot_param_node> -->
-    </plugin>
+      <parameters> $(find cyton_bringup)/config/cyton_controller.yaml </parameters>
+      </plugin>
     </gazebo>
   <ros2_control name="IgnitionSystem" type="system">

File: src/cyton_bringup/urdf/cyton_macros.urdf.xacro (robot description, xacro)
@@ -1,9 +1,11 @@
 <?xml version="1.0"?>
 <robot xmlns:xacro="http://www.ros.org/wiki/xacro">
-    <xacro:include filename="$(find cyton_ros2_gazebo)/urdf/cyton_ignition.xacro" />
-    <!-- <xacro:include filename="$(find cyton_ros2_gazebo)/urdf/cyton_transmission.xacro" /> -->
     <xacro:macro name="cyton_robot">
-        <!-- <xacro:cyton_transmission /> -->
-        <xacro:cyton_ignition />
+        <xacro:if value="$(arg use_sim)">
+            <xacro:cyton_ignition />
+        </xacro:if>
+        <xacro:unless value="$(arg use_sim)">
+            <xacro:cyton_hardware/>
+        </xacro:unless>
         <material name="blue">
           <color rgba= "1 0 0 1"/>
@@ -43,5 +45,5 @@
                 <origin xyz="0 0 0" rpy="0 0 0" />
                 <geometry>
-                    <mesh filename="file://$(find cyton_ros2_gazebo)/meshes/visual/gamma_base.dae" />
+                    <mesh filename="file://$(find cyton_bringup)/meshes/visual/gamma_base.dae" />
                 </geometry>
                 <material name="blue"/>
@@ -50,5 +52,5 @@
                 <origin xyz="0 0 0" rpy="0 0 0" />
                 <geometry>
-                    <mesh filename="file://$(find cyton_ros2_gazebo)/meshes/collision/gamma_base.stl" />
+                    <mesh filename="file://$(find cyton_bringup)/meshes/collision/gamma_base.stl" />
                     <!-- <box size="0.1 0.1 0.007" /> -->
                 </geometry>
@@ -75,5 +77,5 @@
                 <origin xyz="0 0 0" rpy="1.5708 0 3.14159" />
                 <geometry>
-                    <mesh filename="file://$(find cyton_ros2_gazebo)/meshes/visual/joint1.dae" />
+                    <mesh filename="file://$(find cyton_bringup)/meshes/visual/joint1.dae" />
                 </geometry>
                 <material name="blue"/>
@@ -82,5 +84,5 @@
                 <origin xyz="0 0 0" rpy="1.5708 0 3.14159" />
                 <geometry>
-                    <mesh filename="file://$(find cyton_ros2_gazebo)/meshes/collision/joint1.stl" />
+                    <mesh filename="file://$(find cyton_bringup)/meshes/collision/joint1.stl" />
                 </geometry>
             </collision>
@@ -105,5 +107,5 @@
                 <origin xyz="0.028 0 0" rpy="0 1.5708 0" />
                 <geometry>
-                    <mesh filename="file://$(find cyton_ros2_gazebo)/meshes/visual/joint2.dae" />
+                    <mesh filename="file://$(find cyton_bringup)/meshes/visual/joint2.dae" />
                 </geometry>
                 <material name="blue"/>
@@ -112,5 +114,5 @@
                 <origin xyz="0.028 0 0" rpy="0 1.5708 0" />
                 <geometry>
-                    <mesh filename="file://$(find cyton_ros2_gazebo)/meshes/collision/joint2.stl" />
+                    <mesh filename="file://$(find cyton_bringup)/meshes/collision/joint2.stl" />
                 </geometry>
             </collision>
@@ -136,5 +138,5 @@
                 <origin xyz="0 0 0" rpy="0 0 3.92699" />
                 <geometry>
-                    <mesh filename="file://$(find cyton_ros2_gazebo)/meshes/visual/joint3.dae" />
+                    <mesh filename="file://$(find cyton_bringup)/meshes/visual/joint3.dae" />
                 </geometry>
                 <material name="blue"/>
@@ -143,5 +145,5 @@
                 <origin xyz="0 0 0" rpy="0 0 3.92699" />
                 <geometry>
-                    <mesh filename="file://$(find cyton_ros2_gazebo)/meshes/collision/joint3.stl" />
+                    <mesh filename="file://$(find cyton_bringup)/meshes/collision/joint3.stl" />
                     <!-- <sphere radius="0.001" /> -->
                 </geometry>
@@ -168,5 +170,5 @@
                 <origin xyz="0.027 0 0" rpy="1.5708 0 1.5708" />
                 <geometry>
-                    <mesh filename="file://$(find cyton_ros2_gazebo)/meshes/visual/joint4.dae" />
+                    <mesh filename="file://$(find cyton_bringup)/meshes/visual/joint4.dae" />
                 </geometry>
                 <material name="blue"/>
@@ -175,5 +177,5 @@
                 <origin xyz="0.027 0 0" rpy="1.5708 0 1.5708" />
                 <geometry>
-                    <mesh filename="file://$(find cyton_ros2_gazebo)/meshes/collision/joint4.stl" />
+                    <mesh filename="file://$(find cyton_bringup)/meshes/collision/joint4.stl" />
                     <!-- <sphere radius="0.001" /> -->
                 </geometry>
@@ -199,5 +201,5 @@
                 <origin xyz="0 0 0" rpy="1.5708 0 0" />
                 <geometry>
-                    <mesh filename="file://$(find cyton_ros2_gazebo)/meshes/visual/joint5.dae" />
+                    <mesh filename="file://$(find cyton_bringup)/meshes/visual/joint5.dae" />
                 </geometry>
                 <material name="blue"/>
@@ -206,5 +208,5 @@
                 <origin xyz="0 0 0" rpy="1.5708 0 0" />
                 <geometry>
-                    <mesh filename="file://$(find cyton_ros2_gazebo)/meshes/collision/joint5.stl" />
+                    <mesh filename="file://$(find cyton_bringup)/meshes/collision/joint5.stl" />
                     <!-- <sphere radius="0.001" /> -->
                 </geometry>
@@ -230,5 +232,5 @@
                 <origin xyz="0.027 0 0" rpy="1.5708 0 1.5708" />
                 <geometry>
-                    <mesh filename="file://$(find cyton_ros2_gazebo)/meshes/visual/joint6.dae" />
+                    <mesh filename="file://$(find cyton_bringup)/meshes/visual/joint6.dae" />
                 </geometry>
                 <material name="blue"/>
@@ -237,5 +239,5 @@
                 <origin xyz="0.027 0 0" rpy="1.5708 0 1.5708" />
                 <geometry>
-                    <mesh filename="file://$(find cyton_ros2_gazebo)/meshes/collision/joint6.stl" />
+                    <mesh filename="file://$(find cyton_bringup)/meshes/collision/joint6.stl" />
                     <!-- <sphere radius="0.001" /> -->
                 </geometry>
@@ -261,5 +263,5 @@
                 <origin xyz="0 0 0" rpy="0 3.14159 1.5708" />
                 <geometry>
-                    <mesh filename="file://$(find cyton_ros2_gazebo)/meshes/visual/joint7.dae" />
+                    <mesh filename="file://$(find cyton_bringup)/meshes/visual/joint7.dae" />
                 </geometry>
                 <material name="blue"/>
@@ -268,5 +270,5 @@
                 <origin xyz="0 0 0" rpy="0 3.14159 1.5708" />
                 <geometry>
-                    <mesh filename="file://$(find cyton_ros2_gazebo)/meshes/collision/joint7.stl" />
+                    <mesh filename="file://$(find cyton_bringup)/meshes/collision/joint7.stl" />
                     <!-- <sphere radius="0.001" /> -->
                 </geometry>
@@ -300,5 +302,5 @@
                 <origin xyz="0 0 -0.03" rpy="0 0 0" />
                 <geometry>
-                    <mesh filename="file://$(find cyton_ros2_gazebo)/meshes/visual/joint8.dae"/>
+                    <mesh filename="file://$(find cyton_bringup)/meshes/visual/joint8.dae"/>
                 </geometry>
                 <material name="blue"/>
@@ -307,5 +309,5 @@
                 <origin xyz="0 0 -0.03" rpy="0 0 0" />
                 <geometry>
-                    <mesh filename="file://$(find cyton_ros2_gazebo)/meshes/collision/joint8.stl"/>
+                    <mesh filename="file://$(find cyton_bringup)/meshes/collision/joint8.stl"/>
                 </geometry>
             </collision>
@@ -331,5 +333,5 @@
                 <origin xyz="0 0 -0.03" rpy="0 0 0" />
                 <geometry>
-                    <mesh filename="file://$(find cyton_ros2_gazebo)/meshes/visual/joint9.dae"/>
+                    <mesh filename="file://$(find cyton_bringup)/meshes/visual/joint9.dae"/>
                 </geometry>
                 <material name="blue"/>
@@ -338,5 +340,5 @@
                 <origin xyz="0 0 -0.03" rpy="0 0 0" />
                 <geometry>
-                    <mesh filename="file://$(find cyton_ros2_gazebo)/meshes/collision/joint9.stl"/>
+                    <mesh filename="file://$(find cyton_bringup)/meshes/collision/joint9.stl"/>
                 </geometry>
             </collision>

Commit message: simulatin and hardware working

File: src/cyton_bringup/urdf/cyton.hardware.xacro (robot description, xacro)
@@ -1,6 +1,7 @@
 <?xml version="1.0"?>
 <robot xmlns:xacro="http://www.ros.org/wiki/xacro">
-      <xacro:macro name="cyton_hardware">
-        <!-- <xacro:property name="initial_positions" value="${load_yaml(initial_positions_file)['initial_positions']}"/> -->
+      <!-- <xacro:macro name="cyton_hardware"> -->
+      <xacro:macro name="cyton_hardware" params="initial_positions_file">
+      <xacro:property name="initial_positions" value="${xacro.load_yaml(initial_positions_file)['initial_positions']}"/>
         <ros2_control name="DynamixelHardware" type="system">
             <hardware>
@@ -14,5 +15,5 @@
                 <command_interface name="position"/>
                 <state_interface name="position">
-                  <!-- <param name="initial_value">${initial_positions['joint1']}</param> -->
+                  <param name="initial_value">${initial_positions['joint1']}</param>
                 </state_interface>
                 <state_interface name="velocity"/>
@@ -22,5 +23,5 @@
                 <command_interface name="position"/>
                 <state_interface name="position">
-                  <!-- <param name="initial_value">${initial_positions['joint2']}</param> -->
+                  <param name="initial_value">${initial_positions['joint2']}</param>
                 </state_interface>
                 <state_interface name="velocity"/>
@@ -30,5 +31,5 @@
                 <command_interface name="position"/>
                 <state_interface name="position">
-                  <!-- <param name="initial_value">${initial_positions['joint3']}</param> -->
+                  <param name="initial_value">${initial_positions['joint3']}</param>
                 </state_interface>
                 <state_interface name="velocity"/>
@@ -38,5 +39,5 @@
                 <command_interface name="position"/>
                 <state_interface name="position">
-                  <!-- <param name="initial_value">${initial_positions['joint4']}</param> -->
+                  <param name="initial_value">${initial_positions['joint4']}</param>
                 </state_interface>
                 <state_interface name="velocity"/>
@@ -46,5 +47,5 @@
                 <command_interface name="position"/>
                 <state_interface name="position">
-                  <!-- <param name="initial_value">${initial_positions['joint5']}</param> -->
+                  <param name="initial_value">${initial_positions['joint5']}</param>
                 </state_interface>
                 <state_interface name="velocity"/>
@@ -54,5 +55,5 @@
                 <command_interface name="position"/>
                 <state_interface name="position">
-                  <!-- <param name="initial_value">${initial_positions['joint6']}</param> -->
+                  <param name="initial_value">${initial_positions['joint6']}</param>
                 </state_interface>
                 <state_interface name="velocity"/>
@@ -62,5 +63,5 @@
                 <command_interface name="position"/>
                 <state_interface name="position">
-                  <!-- <param name="initial_value">${initial_positions['joint7']}</param> -->
+                  <param name="initial_value">${initial_positions['joint7']}</param>
                 </state_interface>
                 <state_interface name="velocity"/>
@@ -71,5 +72,5 @@
                 <command_interface name="position"/>
                 <state_interface name="position">
-                  <!-- <param name="initial_value">${initial_positions['joint8']}</param> -->
+                  <param name="initial_value">${initial_positions['joint8']}</param>
                 </state_interface>
                 <state_interface name="velocity"/>

File: src/cyton_bringup/urdf/cyton.urdf.xacro (robot description, xacro)
@@ -1,7 +1,7 @@
 <?xml version="1.0"?>
 <robot xmlns:xacro="http://www.ros.org/wiki/xacro" name="cyton">
+  <xacro:arg name="use_sim" default="False"/>
+  <xacro:arg name="initial_positions_file" default="$(find cyton_moveit)/config/initial_positions.yaml" />
   <xacro:include filename="$(find cyton_bringup)/urdf/cyton_macros.urdf.xacro" />
-  <xacro:arg name="use_sim" default="False"/>
-<!-- <xacro:property name="use_sim" value="True"/> -->
   <xacro:if value="$(arg use_sim)">
     <xacro:include filename="$(find cyton_bringup)/urdf/cyton_ignition.xacro" />

File: src/cyton_bringup/urdf/cyton_macros.urdf.xacro (robot description, xacro)
@@ -6,5 +6,5 @@
         </xacro:if>
         <xacro:unless value="$(arg use_sim)">
-            <xacro:cyton_hardware/>
+            <xacro:cyton_hardware initial_positions_file="$(arg initial_positions_file)"/>
         </xacro:unless>
         <material name="blue">
