Commit message: effector size fixed

File: src/cyton_bringup/urdf/cyton.urdf.xacro (robot description, xacro)
@@ -15,5 +15,5 @@
     <parent link="world" />
     <child link = "base_footprint" />
-    <origin xyz="0.0 0.0 0.01" rpy="0.0 0.0 0.0" />
+    <origin xyz="0.0 0.0 0.0001" rpy="0.0 0.0 0.0" />
   </joint>
 </robot>

File: src/cyton_bringup/urdf/cyton_macros.urdf.xacro (robot description, xacro)
@@ -299,14 +299,14 @@
         <link name="link8">
             <visual>
-                <origin xyz="0 0 -0.03" rpy="0 0 0" />
-                <geometry>
-                    <mesh filename="file://$(find cyton_bringup)/meshes/visual/joint8.dae"/>
-                </geometry>
-                <material name="blue"/>
-            </visual>
-            <collision>
-                <origin xyz="0 0 -0.03" rpy="0 0 0" />
-                <geometry>
-                    <mesh filename="file://$(find cyton_bringup)/meshes/collision/joint8.stl"/>
+                <origin xyz="0 0 -0.035" rpy="0 0 3.14" />
+                <geometry>
+                    <mesh filename="file://$(find cyton_bringup)/meshes/visual/joint9_stretched.dae"/>
+                </geometry>
+                <material name="blue"/>
+            </visual>
+            <collision>
+                <origin xyz="0 0 -0.035" rpy="0 0 3.14" />
+                <geometry>
+                    <mesh filename="file://$(find cyton_bringup)/meshes/collision/joint9_stretched.stl"/>
                 </geometry>
             </collision>
@@ -330,14 +330,15 @@
         <link name="link9">
             <visual>
-                <origin xyz="0 0 -0.03" rpy="0 0 0" />
-                <geometry>
-                    <mesh filename="file://$(find cyton_bringup)/meshes/visual/joint9.dae"/>
-                </geometry>
-                <material name="blue"/>
-            </visual>
-            <collision>
-                <origin xyz="0 0 -0.03" rpy="0 0 0" />
-                <geometry>
-                    <mesh filename="file://$(find cyton_bringup)/meshes/collision/joint9.stl"/>
+                <!-- <origin xyz="0 0 -0.03" rpy="0 0 0" /> -->
+                <origin xyz="0 0 -0.035" rpy="0 0 0" />
+                <geometry>
+                    <mesh filename="file://$(find cyton_bringup)/meshes/visual/joint9_stretched.dae"/>
+                </geometry>
+                <material name="blue"/>
+            </visual>
+            <collision>
+                <origin xyz="0 0 -0.035" rpy="0 0 0" />
+                <geometry>
+                    <mesh filename="file://$(find cyton_bringup)/meshes/collision/joint9_stretched.stl"/>
                 </geometry>
             </collision>
