Commit message: working fine

File: src/cyton_bringup/urdf/cyton_macros.urdf.xacro (robot description, xacro)
@@ -286,5 +286,5 @@
             <origin xyz="-0.02131 0.00485 0.077225" rpy="0 0 0" />
             <dynamics damping="0.5" friction="0.5"/>
-            <limit lower="-0.001" upper="0.017" effort="100.0" velocity="1.0" />
+            <limit lower="-0.002" upper="0.018" effort="0.1" velocity="1.0" />
             <axis xyz="1 0 0" />
         </joint>
@@ -324,5 +324,5 @@
             <origin xyz="0.0178 0.00485 0.077225" rpy="0 0 0" />
             <dynamics damping="0.5" friction="0.5"/>
-            <limit lower="-0.017" upper="0.001" effort="100.0" velocity="1.0" />
+            <limit lower="-0.018" upper="0.002" effort="0.1" velocity="1.0" />
             <mimic joint="joint8" multiplier="-1"/>
             <axis xyz="1 0 0" />

Commit message: effort fixed

File: src/cyton_bringup/urdf/cyton_macros.urdf.xacro (robot description, xacro)
@@ -286,5 +286,5 @@
             <origin xyz="-0.02131 0.00485 0.077225" rpy="0 0 0" />
             <dynamics damping="0.5" friction="0.5"/>
-            <limit lower="-0.002" upper="0.018" effort="0.1" velocity="1.0" />
+            <limit lower="-0.002" upper="0.018" effort="100.0" velocity="1.0" />
             <axis xyz="1 0 0" />
         </joint>
@@ -324,5 +324,5 @@
             <origin xyz="0.0178 0.00485 0.077225" rpy="0 0 0" />
             <dynamics damping="0.5" friction="0.5"/>
-            <limit lower="-0.018" upper="0.002" effort="0.1" velocity="1.0" />
+            <limit lower="-0.018" upper="0.002" effort="100.0" velocity="1.0" />
             <mimic joint="joint8" multiplier="-1"/>
             <axis xyz="1 0 0" />

Commit message: meshes and model changed

File: src/cyton_bringup/urdf/cyton_macros.urdf.xacro (robot description, xacro)
@@ -8,6 +8,6 @@
             <xacro:cyton_hardware initial_positions_file="$(arg initial_positions_file)"/>
         </xacro:unless>
-        <material name="blue">
-          <color rgba= "1 0 0 1"/>
+        <material name="TopBlack">
+          <color rgba="0.038 0.038 0.038 1.0"/>
         </material>
         <!-- Initial footprint motor used here -->
@@ -24,5 +24,5 @@
                         <sphere radius="0.001" />
                     </geometry>
-                    <material name="blue"/>
+                    <material name="TopBlack"/>
                 </visual>
                 <collision>
@@ -46,5 +46,5 @@
                     <mesh filename="file://$(find cyton_bringup)/meshes/visual/gamma_base.dae" />
                 </geometry>
-                <material name="blue"/>
+                <material name="TopBlack"/>
             </visual>
             <collision>
@@ -54,8 +54,8 @@
                     <!-- <box size="0.1 0.1 0.007" /> -->
                 </geometry>
-                <material name="blue"/>
-            </collision>
-            <inertial>
-                <mass value="0.2" />
+                <material name="TopBlack"/>
+            </collision>
+            <inertial>
+                <mass value="0.15" />
                 <origin rpy="0 0 0" xyz="0 0 0" />
                 <inertia ixx="1.1027" iyy="1.1027" izz="1.1027"
@@ -76,16 +76,16 @@
                 <origin xyz="0 0 0" rpy="1.5708 0 3.14159" />
                 <geometry>
-                    <mesh filename="file://$(find cyton_bringup)/meshes/visual/joint1.dae" />
-                </geometry>
-                <material name="blue"/>
+                    <mesh filename="file://$(find cyton_bringup)/meshes/visual/link1.dae" />
+                </geometry>
+                <material name="TopBlack"/>
             </visual>
             <collision>
                 <origin xyz="0 0 0" rpy="1.5708 0 3.14159" />
                 <geometry>
-                    <mesh filename="file://$(find cyton_bringup)/meshes/collision/joint1.stl" />
-                </geometry>
-            </collision>
-            <inertial>
-                <mass value="5.0" />
+                    <mesh filename="file://$(find cyton_bringup)/meshes/collision/link1.stl" />
+                </geometry>
+            </collision>
+            <inertial>
+                <mass value="0.15" />
                 <origin rpy="0 0 0" xyz="0 0 0" />
                 <inertia  ixx="0.011208614136379117" ixy="0" ixz="0"
@@ -106,16 +106,16 @@
                 <origin xyz="0.028 0 0" rpy="0 1.5708 0" />
                 <geometry>
-                    <mesh filename="file://$(find cyton_bringup)/meshes/visual/joint2.dae" />
-                </geometry>
-                <material name="blue"/>
+                    <mesh filename="file://$(find cyton_bringup)/meshes/visual/link2.dae" />
+                </geometry>
+                <material name="TopBlack"/>
             </visual>
             <collision>
                 <origin xyz="0.028 0 0" rpy="0 1.5708 0" />
                 <geometry>
-                    <mesh filename="file://$(find cyton_bringup)/meshes/collision/joint2.stl" />
-                </geometry>
-            </collision>
-            <inertial>
-                <mass value="2.0" />
+                    <mesh filename="file://$(find cyton_bringup)/meshes/collision/link2.stl" />
+                </geometry>
+            </collision>
+            <inertial>
+                <mass value="0.15" />
                 <origin rpy="0 0 0" xyz="0 0 0" />
                 <inertia  ixx="0.004978331673653838" ixy="0" ixz="0"
@@ -137,17 +137,17 @@
                 <origin xyz="0 0 0" rpy="0 0 3.92699" />
                 <geometry>
-                    <mesh filename="file://$(find cyton_bringup)/meshes/visual/joint3.dae" />
-                </geometry>
-                <material name="blue"/>
+                    <mesh filename="file://$(find cyton_bringup)/meshes/visual/link3.dae" />
+                </geometry>
+                <material name="TopBlack"/>
             </visual>
             <collision>
                 <origin xyz="0 0 0" rpy="0 0 3.92699" />
                 <geometry>
-                    <mesh filename="file://$(find cyton_bringup)/meshes/collision/joint3.stl" />
-                    <!-- <sphere radius="0.001" /> -->
-                </geometry>
-            </collision>
-            <inertial>
-                <mass value="0.2" />
+                    <mesh filename="file://$(find cyton_bringup)/meshes/collision/link3.stl" />
+                    <!-- <sphere radius="0.001" /> -->
+                </geometry>
+            </collision>
+            <inertial>
+                <mass value="0.15" />
                 <origin rpy="0 0 0" xyz="0 0 0" />
                 <inertia  ixx="0.004185745441913727" ixy="0" ixz="0"
@@ -169,17 +169,17 @@
                 <origin xyz="0.027 0 0" rpy="1.5708 0 1.5708" />
                 <geometry>
-                    <mesh filename="file://$(find cyton_bringup)/meshes/visual/joint4.dae" />
-                </geometry>
-                <material name="blue"/>
+                    <mesh filename="file://$(find cyton_bringup)/meshes/visual/link4.dae" />
+                </geometry>
+                <material name="TopBlack"/>
             </visual>
             <collision>
                 <origin xyz="0.027 0 0" rpy="1.5708 0 1.5708" />
                 <geometry>
-                    <mesh filename="file://$(find cyton_bringup)/meshes/collision/joint4.stl" />
-                    <!-- <sphere radius="0.001" /> -->
-                </geometry>
-            </collision>
-            <inertial>
-                <mass value="0.2" />
+                    <mesh filename="file://$(find cyton_bringup)/meshes/collision/link4.stl" />
+                    <!-- <sphere radius="0.001" /> -->
+                </geometry>
+            </collision>
+            <inertial>
+                <mass value="0.15" />
                 <origin rpy="0 0 0" xyz="0 0 0" />
                 <inertia  ixx="0.0002991427484832406" ixy="0" ixz="0"
@@ -200,17 +200,17 @@
                 <origin xyz="0 0 0" rpy="1.5708 0 0" />
                 <geometry>
-                    <mesh filename="file://$(find cyton_bringup)/meshes/visual/joint5.dae" />
-                </geometry>
-                <material name="blue"/>
+                    <mesh filename="file://$(find cyton_bringup)/meshes/visual/link5.dae" />
+                </geometry>
+                <material name="TopBlack"/>
             </visual>
             <collision>
                 <origin xyz="0 0 0" rpy="1.5708 0 0" />
                 <geometry>
-                    <mesh filename="file://$(find cyton_bringup)/meshes/collision/joint5.stl" />
-                    <!-- <sphere radius="0.001" /> -->
-                </geometry>
-            </collision>
-            <inertial>
-                <mass value="0.2" />
+                    <mesh filename="file://$(find cyton_bringup)/meshes/collision/link5.stl" />
+                    <!-- <sphere radius="0.001" /> -->
+                </geometry>
+            </collision>
+            <inertial>
+                <mass value="0.15" />
                 <origin rpy="0 0 0" xyz="0 0 0" />
                 <inertia  ixx="0.004619866095305994" ixy="0" ixz="0"
@@ -231,17 +231,17 @@
                 <origin xyz="0.027 0 0" rpy="1.5708 0 1.5708" />
                 <geometry>
-                    <mesh filename="file://$(find cyton_bringup)/meshes/visual/joint6.dae" />
-                </geometry>
-                <material name="blue"/>
+                    <mesh filename="file://$(find cyton_bringup)/meshes/visual/link6.dae" />
+                </geometry>
+                <material name="TopBlack"/>
             </visual>
             <collision>
                 <origin xyz="0.027 0 0" rpy="1.5708 0 1.5708" />
                 <geometry>
-                    <mesh filename="file://$(find cyton_bringup)/meshes/collision/joint6.stl" />
-                    <!-- <sphere radius="0.001" /> -->
-                </geometry>
-            </collision>
-            <inertial>
-                <mass value="0.2" />
+                    <mesh filename="file://$(find cyton_bringup)/meshes/collision/link6.stl" />
+                    <!-- <sphere radius="0.001" /> -->
+                </geometry>
+            </collision>
+            <inertial>
+                <mass value="0.15" />
                 <origin rpy="0 0 0" xyz="0 0 0" />
                 <inertia  ixx="0.002306163215052582" ixy="0" ixz="0"
@@ -262,17 +262,17 @@
                 <origin xyz="0 0 0" rpy="0 3.14159 1.5708" />
                 <geometry>
-                    <mesh filename="file://$(find cyton_bringup)/meshes/visual/joint7.dae" />
-                </geometry>
-                <material name="blue"/>
+                    <mesh filename="file://$(find cyton_bringup)/meshes/visual/link7.dae" />
+                </geometry>
+                <material name="TopBlack"/>
             </visual>
             <collision>
                 <origin xyz="0 0 0" rpy="0 3.14159 1.5708" />
                 <geometry>
-                    <mesh filename="file://$(find cyton_bringup)/meshes/collision/joint7.stl" />
-                    <!-- <sphere radius="0.001" /> -->
-                </geometry>
-            </collision>
-            <inertial>
-                <mass value="0.2" />
+                    <mesh filename="file://$(find cyton_bringup)/meshes/collision/link7.stl" />
+                    <!-- <sphere radius="0.001" /> -->
+                </geometry>
+            </collision>
+            <inertial>
+                <mass value="0.15" />
                 <origin rpy="0 0 0" xyz="0 0 0" />
                 <inertia  ixx="0.0015572863522148085" ixy="0" ixz="0"
@@ -299,14 +299,14 @@
         <link name="link8">
             <visual>
-                <origin xyz="0 0 -0.035" rpy="0 0 3.14" />
-                <geometry>
-                    <mesh filename="file://$(find cyton_bringup)/meshes/visual/joint9_stretched.dae"/>
-                </geometry>
-                <material name="blue"/>
-            </visual>
-            <collision>
-                <origin xyz="0 0 -0.035" rpy="0 0 3.14" />
-                <geometry>
-                    <mesh filename="file://$(find cyton_bringup)/meshes/collision/joint9_stretched.stl"/>
+                <origin xyz="0 0.0 -0.035" rpy="0 0 0" />
+                <geometry>
+                    <mesh filename="file://$(find cyton_bringup)/meshes/visual/link8.dae" scale="1.0 1.0 2.0"/>
+                </geometry>
+                <material name="TopBlack"/>
+            </visual>
+            <collision>
+                <origin xyz="0 0.0 -0.035" rpy="0 0 0" />
+                <geometry>
+                    <mesh filename="file://$(find cyton_bringup)/meshes/collision/link8.stl" scale="1.0 1.0 2.0"/>
                 </geometry>
             </collision>
@@ -330,15 +330,14 @@
         <link name="link9">
             <visual>
-                <!-- <origin xyz="0 0 -0.03" rpy="0 0 0" /> -->
                 <origin xyz="0 0 -0.035" rpy="0 0 0" />
                 <geometry>
-                    <mesh filename="file://$(find cyton_bringup)/meshes/visual/joint9_stretched.dae"/>
-                </geometry>
-                <material name="blue"/>
+                    <mesh filename="file://$(find cyton_bringup)/meshes/visual/link9.dae" scale="1.0 1.0 2.0"/>
+                </geometry>
+                <material name="TopBlack"/>
             </visual>
             <collision>
                 <origin xyz="0 0 -0.035" rpy="0 0 0" />
                 <geometry>
-                    <mesh filename="file://$(find cyton_bringup)/meshes/collision/joint9_stretched.stl"/>
+                    <mesh filename="file://$(find cyton_bringup)/meshes/collision/link9.stl" scale="1.0 1.0 2.0"/>
                 </geometry>
             </collision>

Commit message: worlds edited

File: src/cyton_bringup/urdf/cyton_macros.urdf.xacro (robot description, xacro)
@@ -299,14 +299,14 @@
         <link name="link8">
             <visual>
-                <origin xyz="0 0.0 -0.035" rpy="0 0 0" />
-                <geometry>
-                    <mesh filename="file://$(find cyton_bringup)/meshes/visual/link8.dae" scale="1.0 1.0 2.0"/>
-                </geometry>
-                <material name="TopBlack"/>
-            </visual>
-            <collision>
-                <origin xyz="0 0.0 -0.035" rpy="0 0 0" />
-                <geometry>
-                    <mesh filename="file://$(find cyton_bringup)/meshes/collision/link8.stl" scale="1.0 1.0 2.0"/>
+                <origin xyz="0 0.0 -0.04" rpy="0 0 0" />
+                <geometry>
+                    <mesh filename="file://$(find cyton_bringup)/meshes/visual/link8.dae" scale="1.0 1.0 2.2"/>
+                </geometry>
+                <material name="TopBlack"/>
+            </visual>
+            <collision>
+                <origin xyz="0 0.0 -0.04" rpy="0 0 0" />
+                <geometry>
+                    <mesh filename="file://$(find cyton_bringup)/meshes/collision/link8.stl" scale="1.0 1.0 2.2"/>
                 </geometry>
             </collision>
@@ -330,14 +330,14 @@
         <link name="link9">
             <visual>
-                <origin xyz="0 0 -0.035" rpy="0 0 0" />
-                <geometry>
-                    <mesh filename="file://$(find cyton_bringup)/meshes/visual/link9.dae" scale="1.0 1.0 2.0"/>
-                </geometry>
-                <material name="TopBlack"/>
-            </visual>
-            <collision>
-                <origin xyz="0 0 -0.035" rpy="0 0 0" />
-                <geometry>
-                    <mesh filename="file://$(find cyton_bringup)/meshes/collision/link9.stl" scale="1.0 1.0 2.0"/>
+                <origin xyz="0 0 -0.04" rpy="0 0 0" />
+                <geometry>
+                    <mesh filename="file://$(find cyton_bringup)/meshes/visual/link9.dae" scale="1.0 1.0 2.2"/>
+                </geometry>
+                <material name="TopBlack"/>
+            </visual>
+            <collision>
+                <origin xyz="0 0 -0.04" rpy="0 0 0" />
+                <geometry>
+                    <mesh filename="file://$(find cyton_bringup)/meshes/collision/link9.stl" scale="1.0 1.0 2.2"/>
                 </geometry>
             </collision>
