Commit message: split cyton into two packages

File: src/cyton_description/urdf/cyton.urdf.xacro (robot description, xacro)
@@ -3,10 +3,10 @@
   <xacro:arg name="use_sim" default="False"/>
   <xacro:arg name="initial_positions_file" default="$(find cyton_moveit)/config/initial_positions.yaml" />
-  <xacro:include filename="$(find cyton_bringup)/urdf/cyton_macros.urdf.xacro" />
+  <xacro:include filename="$(find cyton_description)/urdf/cyton_macros.urdf.xacro" />
   <xacro:if value="$(arg use_sim)">
-    <xacro:include filename="$(find cyton_bringup)/urdf/cyton_ignition.xacro" />
+    <xacro:include filename="$(find cyton_description)/urdf/cyton_ignition.xacro" />
   </xacro:if>
   <xacro:unless value="$(arg use_sim)">
-    <xacro:include filename="$(find cyton_bringup)/urdf/cyton.hardware.xacro" />
+    <xacro:include filename="$(find cyton_description)/urdf/cyton.hardware.xacro" />
   </xacro:unless>
   <xacro:cyton_robot/>

File: src/cyton_description/urdf/cyton_macros.urdf.xacro (robot description, xacro)
@@ -44,5 +44,5 @@
                 <origin xyz="0 0 0" rpy="0 0 0" />
                 <geometry>
-                    <mesh filename="file://$(find cyton_bringup)/meshes/visual/gamma_base.dae" />
+                    <mesh filename="file://$(find cyton_description)/meshes/visual/gamma_base.dae" />
                 </geometry>
                 <material name="blue"/>
@@ -51,5 +51,5 @@
                 <origin xyz="0 0 0" rpy="0 0 0" />
                 <geometry>
-                    <mesh filename="file://$(find cyton_bringup)/meshes/collision/gamma_base.stl" />
+                    <mesh filename="file://$(find cyton_description)/meshes/collision/gamma_base.stl" />
                     <!-- <box size="0.1 0.1 0.007" /> -->
                 </geometry>
@@ -76,5 +76,5 @@
                 <origin xyz="0 0 0" rpy="1.5708 0 3.14159" />
                 <geometry>
-                    <mesh filename="file://$(find cyton_bringup)/meshes/visual/joint1.dae" />
+                    <mesh filename="file://$(find cyton_description)/meshes/visual/joint1.dae" />
                 </geometry>
                 <material name="blue"/>
@@ -83,5 +83,5 @@
                 <origin xyz="0 0 0" rpy="1.5708 0 3.14159" />
                 <geometry>
-                    <mesh filename="file://$(find cyton_bringup)/meshes/collision/joint1.stl" />
+                    <mesh filename="file://$(find cyton_description)/meshes/collision/joint1.stl" />
                 </geometry>
             </collision>
@@ -106,5 +106,5 @@
                 <origin xyz="0.028 0 0" rpy="0 1.5708 0" />
                 <geometry>
-                    <mesh filename="file://$(find cyton_bringup)/meshes/visual/joint2.dae" />
+                    <mesh filename="file://$(find cyton_description)/meshes/visual/joint2.dae" />
                 </geometry>
                 <material name="blue"/>
@@ -113,5 +113,5 @@
                 <origin xyz="0.028 0 0" rpy="0 1.5708 0" />
                 <geometry>
-                    <mesh filename="file://$(find cyton_bringup)/meshes/collision/joint2.stl" />
+                    <mesh filename="file://$(find cyton_description)/meshes/collision/joint2.stl" />
                 </geometry>
             </collision>
@@ -137,5 +137,5 @@
                 <origin xyz="0 0 0" rpy="0 0 3.92699" />
                 <geometry>
-                    <mesh filename="file://$(find cyton_bringup)/meshes/visual/joint3.dae" />
+                    <mesh filename="file://$(find cyton_description)/meshes/visual/joint3.dae" />
                 </geometry>
                 <material name="blue"/>
@@ -144,5 +144,5 @@
                 <origin xyz="0 0 0" rpy="0 0 3.92699" />
                 <geometry>
-                    <mesh filename="file://$(find cyton_bringup)/meshes/collision/joint3.stl" />
+                    <mesh filename="file://$(find cyton_description)/meshes/collision/joint3.stl" />
                     <!-- <sphere radius="0.001" /> -->
                 </geometry>
@@ -169,5 +169,5 @@
                 <origin xyz="0.027 0 0" rpy="1.5708 0 1.5708" />
                 <geometry>
-                    <mesh filename="file://$(find cyton_bringup)/meshes/visual/joint4.dae" />
+                    <mesh filename="file://$(find cyton_description)/meshes/visual/joint4.dae" />
                 </geometry>
                 <material name="blue"/>
@@ -176,5 +176,5 @@
                 <origin xyz="0.027 0 0" rpy="1.5708 0 1.5708" />
                 <geometry>
-                    <mesh filename="file://$(find cyton_bringup)/meshes/collision/joint4.stl" />
+                    <mesh filename="file://$(find cyton_description)/meshes/collision/joint4.stl" />
                     <!-- <sphere radius="0.001" /> -->
                 </geometry>
@@ -200,5 +200,5 @@
                 <origin xyz="0 0 0" rpy="1.5708 0 0" />
                 <geometry>
-                    <mesh filename="file://$(find cyton_bringup)/meshes/visual/joint5.dae" />
+                    <mesh filename="file://$(find cyton_description)/meshes/visual/joint5.dae" />
                 </geometry>
                 <material name="blue"/>
@@ -207,5 +207,5 @@
                 <origin xyz="0 0 0" rpy="1.5708 0 0" />
                 <geometry>
-                    <mesh filename="file://$(find cyton_bringup)/meshes/collision/joint5.stl" />
+                    <mesh filename="file://$(find cyton_description)/meshes/collision/joint5.stl" />
                     <!-- <sphere radius="0.001" /> -->
                 </geometry>
@@ -231,5 +231,5 @@
                 <origin xyz="0.027 0 0" rpy="1.5708 0 1.5708" />
                 <geometry>
-                    <mesh filename="file://$(find cyton_bringup)/meshes/visual/joint6.dae" />
+                    <mesh filename="file://$(find cyton_description)/meshes/visual/joint6.dae" />
                 </geometry>
                 <material name="blue"/>
@@ -238,5 +238,5 @@
                 <origin xyz="0.027 0 0" rpy="1.5708 0 1.5708" />
                 <geometry>
-                    <mesh filename="file://$(find cyton_bringup)/meshes/collision/joint6.stl" />
+                    <mesh filename="file://$(find cyton_description)/meshes/collision/joint6.stl" />
                     <!-- <sphere radius="0.001" /> -->
                 </geometry>
@@ -262,5 +262,5 @@
                 <origin xyz="0 0 0" rpy="0 3.14159 1.5708" />
                 <geometry>
-                    <mesh filename="file://$(find cyton_bringup)/meshes/visual/joint7.dae" />
+                    <mesh filename="file://$(find cyton_description)/meshes/visual/joint7.dae" />
                 </geometry>
                 <material name="blue"/>
@@ -269,5 +269,5 @@
                 <origin xyz="0 0 0" rpy="0 3.14159 1.5708" />
                 <geometry>
-                    <mesh filename="file://$(find cyton_bringup)/meshes/collision/joint7.stl" />
+                    <mesh filename="file://$(find cyton_description)/meshes/collision/joint7.stl" />
                     <!-- <sphere radius="0.001" /> -->
                 </geometry>
@@ -301,5 +301,5 @@
                 <origin xyz="0 0 -0.035" rpy="0 0 3.14" />
                 <geometry>
-                    <mesh filename="file://$(find cyton_bringup)/meshes/visual/joint9_stretched.dae"/>
+                    <mesh filename="file://$(find cyton_description)/meshes/visual/joint9_stretched.dae"/>
                 </geometry>
                 <material name="blue"/>
@@ -308,5 +308,5 @@
                 <origin xyz="0 0 -0.035" rpy="0 0 3.14" />
                 <geometry>
-                    <mesh filename="file://$(find cyton_bringup)/meshes/collision/joint9_stretched.stl"/>
+                    <mesh filename="file://$(find cyton_description)/meshes/collision/joint9_stretched.stl"/>
                 </geometry>
             </collision>
@@ -333,5 +333,5 @@
                 <origin xyz="0 0 -0.035" rpy="0 0 0" />
                 <geometry>
-                    <mesh filename="file://$(find cyton_bringup)/meshes/visual/joint9_stretched.dae"/>
+                    <mesh filename="file://$(find cyton_description)/meshes/visual/joint9_stretched.dae"/>
                 </geometry>
                 <material name="blue"/>
@@ -340,5 +340,5 @@
                 <origin xyz="0 0 -0.035" rpy="0 0 0" />
                 <geometry>
-                    <mesh filename="file://$(find cyton_bringup)/meshes/collision/joint9_stretched.stl"/>
+                    <mesh filename="file://$(find cyton_description)/meshes/collision/joint9_stretched.stl"/>
                 </geometry>
             </collision>
