Commit message: work in progress

File: src/mobile_arm_description/description/cyton/cyton_macros.urdf.xacro (robot description, xacro)
@@ -44,5 +44,5 @@
                 <origin xyz="0 0 0" rpy="0 0 0" />
                 <geometry>
-                    <mesh filename="file://$(find cyton_description)/meshes/visual/gamma_base.dae" />
+                    <mesh filename="file://$(arg models_dir)/cyton/meshes/visual/gamma_base.dae" />
                 </geometry>
                 <material name="blue"/>
@@ -51,5 +51,5 @@
                 <origin xyz="0 0 0" rpy="0 0 0" />
                 <geometry>
-                    <mesh filename="file://$(find cyton_description)/meshes/collision/gamma_base.stl" />
+                    <mesh filename="file://$(arg models_dir)/cyton/meshes/collision/gamma_base.stl" />
                     <!-- <box size="0.1 0.1 0.007" /> -->
                 </geometry>
@@ -76,5 +76,5 @@
                 <origin xyz="0 0 0" rpy="1.5708 0 3.14159" />
                 <geometry>
-                    <mesh filename="file://$(find cyton_description)/meshes/visual/joint1.dae" />
+                    <mesh filename="file://$(arg models_dir)/cyton/meshes/visual/joint1.dae" />
                 </geometry>
                 <material name="blue"/>
@@ -83,5 +83,5 @@
                 <origin xyz="0 0 0" rpy="1.5708 0 3.14159" />
                 <geometry>
-                    <mesh filename="file://$(find cyton_description)/meshes/collision/joint1.stl" />
+                    <mesh filename="file://$(arg models_dir)/cyton/meshes/collision/joint1.stl" />
                 </geometry>
             </collision>
@@ -106,5 +106,5 @@
                 <origin xyz="0.028 0 0" rpy="0 1.5708 0" />
                 <geometry>
-                    <mesh filename="file://$(find cyton_description)/meshes/visual/joint2.dae" />
+                    <mesh filename="file://$(arg models_dir)/cyton/meshes/visual/joint2.dae" />
                 </geometry>
                 <material name="blue"/>
@@ -113,5 +113,5 @@
                 <origin xyz="0.028 0 0" rpy="0 1.5708 0" />
                 <geometry>
-                    <mesh filename="file://$(find cyton_description)/meshes/collision/joint2.stl" />
+                    <mesh filename="file://$(arg models_dir)/cyton/meshes/collision/joint2.stl" />
                 </geometry>
             </collision>
@@ -137,5 +137,5 @@
                 <origin xyz="0 0 0" rpy="0 0 3.92699" />
                 <geometry>
-                    <mesh filename="file://$(find cyton_description)/meshes/visual/joint3.dae" />
+                    <mesh filename="file://$(arg models_dir)/cyton/meshes/visual/joint3.dae" />
                 </geometry>
                 <material name="blue"/>
@@ -144,5 +144,5 @@
                 <origin xyz="0 0 0" rpy="0 0 3.92699" />
                 <geometry>
-                    <mesh filename="file://$(find cyton_description)/meshes/collision/joint3.stl" />
+                    <mesh filename="file://$(arg models_dir)/cyton/meshes/collision/joint3.stl" />
                     <!-- <sphere radius="0.001" /> -->
                 </geometry>
@@ -169,5 +169,5 @@
                 <origin xyz="0.027 0 0" rpy="1.5708 0 1.5708" />
                 <geometry>
-                    <mesh filename="file://$(find cyton_description)/meshes/visual/joint4.dae" />
+                    <mesh filename="file://$(arg models_dir)/cyton/meshes/visual/joint4.dae" />
                 </geometry>
                 <material name="blue"/>
@@ -176,5 +176,5 @@
                 <origin xyz="0.027 0 0" rpy="1.5708 0 1.5708" />
                 <geometry>
-                    <mesh filename="file://$(find cyton_description)/meshes/collision/joint4.stl" />
+                    <mesh filename="file://$(arg models_dir)/cyton/meshes/collision/joint4.stl" />
                     <!-- <sphere radius="0.001" /> -->
                 </geometry>
@@ -200,5 +200,5 @@
                 <origin xyz="0 0 0" rpy="1.5708 0 0" />
                 <geometry>
-                    <mesh filename="file://$(find cyton_description)/meshes/visual/joint5.dae" />
+                    <mesh filename="file://$(arg models_dir)/cyton/meshes/visual/joint5.dae" />
                 </geometry>
                 <material name="blue"/>
@@ -207,5 +207,5 @@
                 <origin xyz="0 0 0" rpy="1.5708 0 0" />
                 <geometry>
-                    <mesh filename="file://$(find cyton_description)/meshes/collision/joint5.stl" />
+                    <mesh filename="file://$(arg models_dir)/cyton/meshes/collision/joint5.stl" />
                     <!-- <sphere radius="0.001" /> -->
                 </geometry>
@@ -231,5 +231,5 @@
                 <origin xyz="0.027 0 0" rpy="1.5708 0 1.5708" />
                 <geometry>
-                    <mesh filename="file://$(find cyton_description)/meshes/visual/joint6.dae" />
+                    <mesh filename="file://$(arg models_dir)/cyton/meshes/visual/joint6.dae" />
                 </geometry>
                 <material name="blue"/>
@@ -238,5 +238,5 @@
                 <origin xyz="0.027 0 0" rpy="1.5708 0 1.5708" />
                 <geometry>
-                    <mesh filename="file://$(find cyton_description)/meshes/collision/joint6.stl" />
+                    <mesh filename="file://$(arg models_dir)/cyton/meshes/collision/joint6.stl" />
                     <!-- <sphere radius="0.001" /> -->
                 </geometry>
@@ -262,5 +262,5 @@
                 <origin xyz="0 0 0" rpy="0 3.14159 1.5708" />
                 <geometry>
-                    <mesh filename="file://$(find cyton_description)/meshes/visual/joint7.dae" />
+                    <mesh filename="file://$(arg models_dir)/cyton/meshes/visual/joint7.dae" />
                 </geometry>
                 <material name="blue"/>
@@ -269,5 +269,5 @@
                 <origin xyz="0 0 0" rpy="0 3.14159 1.5708" />
                 <geometry>
-                    <mesh filename="file://$(find cyton_description)/meshes/collision/joint7.stl" />
+                    <mesh filename="file://$(arg models_dir)/cyton/meshes/collision/joint7.stl" />
                     <!-- <sphere radius="0.001" /> -->
                 </geometry>
@@ -301,5 +301,5 @@
                 <origin xyz="0 0 -0.035" rpy="0 0 3.14" />
                 <geometry>
-                    <mesh filename="file://$(find cyton_description)/meshes/visual/joint9_stretched.dae"/>
+                    <mesh filename="file://$(arg models_dir)/cyton/meshes/visual/joint9_stretched.dae"/>
                 </geometry>
                 <material name="blue"/>
@@ -308,5 +308,5 @@
                 <origin xyz="0 0 -0.035" rpy="0 0 3.14" />
                 <geometry>
-                    <mesh filename="file://$(find cyton_description)/meshes/collision/joint9_stretched.stl"/>
+                    <mesh filename="file://$(arg models_dir)/cyton/meshes/collision/joint9_stretched.stl"/>
                 </geometry>
             </collision>
@@ -333,5 +333,5 @@
                 <origin xyz="0 0 -0.035" rpy="0 0 0" />
                 <geometry>
-                    <mesh filename="file://$(find cyton_description)/meshes/visual/joint9_stretched.dae"/>
+                    <mesh filename="file://$(arg models_dir)/cyton/meshes/visual/joint9_stretched.dae"/>
                 </geometry>
                 <material name="blue"/>
@@ -340,5 +340,5 @@
                 <origin xyz="0 0 -0.035" rpy="0 0 0" />
                 <geometry>
-                    <mesh filename="file://$(find cyton_description)/meshes/collision/joint9_stretched.stl"/>
+                    <mesh filename="file://$(arg models_dir)/cyton/meshes/collision/joint9_stretched.stl"/>
                 </geometry>
             </collision>

File: src/mobile_arm_description/description/pioneer3dx/main.xacro (robot description, xacro)
@@ -1,7 +1,8 @@
 <?xml version="1.0"?>
 <robot xmlns:xacro="http://ros.org/wiki/xacro" name="pioneer3dx" >
-  <xacro:arg name="models_dir"       default="$(find pioneer_description)/description"/>
+  <xacro:arg name="models_dir"       default="$(find mobile_arm_description)/description"/>
   <xacro:arg name="robot_model"      default="pioneer3dx"/>
   <xacro:arg name="laser_model"      default="hokuyo"/>
+  <xacro:arg name="arm_model"        default="cyton"/>
   <xacro:arg name="namespace"        default="r0"/>
   <xacro:arg name="robot_name"       default="r0"/>
@@ -9,9 +10,10 @@
   <xacro:arg name="laser0_visualize" default="true"/>
   <xacro:arg name="laser0_driver"    default="gpu"/>
-  <!-- <xacro:arg name="use_sim"          default="False"/> -->
+  <xacro:arg name="use_sim"          default="false"/>
   <xacro:property name="models_dir"    value="$(arg models_dir)"/>
   <xacro:property name="namespace"    value="$(arg namespace)"/>
   <xacro:property name="robot_model"   value="$(arg robot_model)"/>
   <xacro:property name="laser_model"   value="$(arg laser_model)"/>
+  <xacro:property name="arm_model"   value="$(arg arm_model)"/>
   <!-- Import Rviz colors -->
   <xacro:include filename="${models_dir}/materials.xacro" />
@@ -26,6 +28,6 @@
   <xacro:include filename="${models_dir}/${laser_model}/main.xacro"/>
   <xacro:laser name="laser0" parent="top" namespace="${namespace}" topic_name="$(arg laser0_topic)" frame_name="laser0" xyz="0.15 0.0 0.06" rpy="0 0 0" driver="$(arg laser0_driver)" visualize="$(arg laser0_visualize)"/>
-  <!-- Cyton arm -->
-  <!-- <xacro:include filename="$(find cyton_bringup)/urdf/cyton.urdf.xacro" />
-  <xacro:cyton use_sim="$(use_sim)"/> -->
+  <!-- Arm -->
+  <xacro:include filename="${models_dir}/${arm_model}/urdf/main.xacro" />
+  <xacro:arm name="cyton" parent="top" xyz="0.0 0.0 0.0" rpy="0 0 0" use_sim="$(use_sim)"/>
 </robot>
